File: CG Files.kicad_pcb (KiCad board)
At the start: 4 copper layers, 296 parts, among them Y1 Crystal_GND24

Commit message: finished routing
//TODO
-> add mechanical support
-> daughter board
-> recheck nodes/conections
-> silk screen
Parts:
- removed BUF7, BUF9: 74AHC1G125, Package_TO_SOT_SMD:SOT-553
- removed C101, C102, C103, C105, C108, C111, C90, C91, C93, C99: .1uF, Capacitor_SMD:C_0402_1005Metric
- removed the C88 at (237.9, 132.6)
- removed the C94 at (238.1, 139.1)
- removed the C96 at (204.4, 129.2)
- removed the C97 at (205.4, 121.2)
- removed the C98 at (204.3, 146.4)
- removed D6, D7: ESD9X5.0ST5G, Diode_SMD:D_SOD-923
- removed INV7: 74LVC1GU04DRLR, Package_TO_SOT_SMD:SOT-553
- removed LS2: TXS0102DCUR, Package_SO:VSSOP-8_2.3x2mm_P0.5mm
- removed the R64 at (123.5, 138.5)
- removed the R65 at (145.8, 105.3)
- removed the R83 at (208.1, 124.1)
- removed the R84 at (211.5, 125.0)
- added R81: 100, Resistor_SMD:R_0603_1608Metric, F.Cu at (53.2, 130.1)
- R62: value 100 -> 10k
- R63: value 22 -> 100
- moved LD2 203.9 mm to (80.5, 69.5), turned to 180 degrees
- moved R67 197.7 mm to (104.2, 35.1), turned to 0 degrees
- moved C76 197.0 mm to (83.5, 71.3), turned to -90 degrees
- moved SPST2 193.2 mm to (103.3, 37.7), turned to 0 degrees
- moved AND3 189.4 mm to (88.6, 66.4), turned to -90 degrees
- moved C87 188.7 mm to (90.0, 69.2), turned to 0 degrees
- moved R66 188.6 mm to (88.3, 58.8), turned to 180 degrees
- moved C79 185.9 mm to (85.2, 60.2)
- moved LD5 185.9 mm to (88.3, 61.9)
- moved SPST1 184.4 mm to (89.0, 56.1)
- moved C82 183.7 mm to (86.7, 51.3)
- moved R77 182.8 mm to (101.5, 53.7), turned to 90 degrees
- moved R80 182.5 mm to (107.4, 54.9), turned to 90 degrees
- moved LD4 182.5 mm to (82.0, 64.0)
- moved C78 182.4 mm to (79.1, 62.3)
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- renumbered 1V8 to 1V1, 3V3 to 3V1, BUCK_1V8 to BUCK_1V1, BUCK_3V8 to BUCK_3V1, C12 to C11, C13 to C12, C11 to C13, C89 to C88, C92 to C89, C100 to C92, C104 to C94, C107 to C96, C109 to C97, C110 to C98, EFUSE to EFUSE1, R66 to R64, R67 to R65, R68 to R66, R69 to R67, R70 to R68, R71 to R69, R72 to R70, R73 to R71, R74 to R72, R75 to R73, R76 to R74, R77 to R75, R78 to R76, R79 to R77, R80 to R78, R81 to R79, R82 to R80, R85 to R83, R86 to R84, R87 to R85, R88 to R86, R89 to R87, R90 to R88, R91 to R89, R92 to R90, R93 to R91, TRGT_PWR_EN to TRGT_PWR_ON1, VTGT_1V8 to VTGT_1V1, VTGT_3V3 to VTGT_3V1
Connections:
- BUF11 pad 4: /Profile_Switching/LQFP100_PIN_34 -> /Profile_Switching/LQFP100_PIN_69
- BUF13 pad 2: /Profile_Switching/LQFP100_PIN_33 -> /Profile_Switching/LQFP100_PIN_68
- DEC1 pad 6: MCU_TARGET_PROFILE_ENABLE -> Net-(DEC1-G1)
- J_CARDX_L_1 pad 01: /Profile_Switching/LQFP64_PIN_47 -> unconnected-(J_CARDX_L_1-Pad01)
- J_CARDX_L_1 pad 02: TARGET_PWR_ENABLE -> unconnected-(J_CARDX_L_1-Pad02)
- J_CARDX_L_1 pad 03: unconnected-(J_CARDX_L_1-Pad03) -> LQFP100_ENABLE
- J_CARDX_L_1 pad 05: unconnected-(J_CARDX_L_1-Pad05) -> LQFP64_ENABLE
- J_CARDX_L_1 pad 07: TARGET_POWER_SUPPLY -> unconnected-(J_CARDX_L_1-Pad07)
- J_CARDX_L_1 pad 08: unconnected-(J_CARDX_L_1-Pad08) -> /Profile_Switching/LQFP100_PIN_27
- J_CARDX_L_1 pad 101: TARGET_POWER_SUPPLY -> unconnected-(J_CARDX_L_1-Pad101)
- J_CARDX_L_1 pad 102: TARGET_POWER_SUPPLY -> unconnected-(J_CARDX_L_1-Pad102)
- J_CARDX_L_1 pad 105: TARGET_POWER_SUPPLY -> unconnected-(J_CARDX_L_1-Pad105)
- J_CARDX_L_1 pad 108: TARGET_POWER_SUPPLY -> unconnected-(J_CARDX_L_1-Pad108)
- J_CARDX_L_1 pad 109: TARGET_POWER_SUPPLY -> /Profile_Switching/LQFP64_PIN_19
- J_CARDX_L_1 pad 113: /Profile_Switching/LQFP100_PIN_22 -> /Profile_Switching/LQFP64_PIN_48
- J_CARDX_L_1 pad 114: /Profile_Switching/LQFP64_PIN_19 -> unconnected-(J_CARDX_L_1-Pad114)
- J_CARDX_L_1 pad 115: unconnected-(J_CARDX_L_1-Pad115) -> /Profile_Switching/LQFP100_PIN_69
- J_CARDX_L_1 pad 117: unconnected-(J_CARDX_L_1-Pad117) -> /Profile_Switching/LQFP64_PIN_42
- J_CARDX_L_1 pad 118: unconnected-(J_CARDX_L_1-Pad118) -> /Profile_Switching/LQFP100_PIN_22
- J_CARDX_L_1 pad 119: /Profile_Switching/LQFP64_PIN_48 -> /Profile_Switching/LQFP64_PIN_7
- J_CARDX_L_1 pad 12: /Profile_Switching/LQFP100_PIN_10 -> unconnected-(J_CARDX_L_1-Pad12)
- J_CARDX_L_1 pad 120: TARGET_POWER_SUPPLY -> /Profile_Switching/LQFP64_PIN_60
- J_CARDX_L_1 pad 18: /Profile_Switching/LQFP100_PIN_27 -> unconnected-(J_CARDX_L_1-Pad18)
- J_CARDX_L_1 pad 25: LQFP64_ENABLE -> unconnected-(J_CARDX_L_1-Pad25)
- J_CARDX_L_1 pad 27: LQFP100_ENABLE -> unconnected-(J_CARDX_L_1-Pad27)
- J_CARDX_L_1 pad 35: /Profile_Switching/LQFP100_PIN_68 -> unconnected-(J_CARDX_L_1-Pad35)
- J_CARDX_L_1 pad 37: /Profile_Switching/LQFP100_PIN_69 -> /Profile_Switching/LQFP64_PIN_43
- J_CARDX_L_1 pad 40: unconnected-(J_CARDX_L_1-Pad40) -> /Profile_Switching/LQFP100_PIN_94
- J_CARDX_L_1 pad 45: /Profile_Switching/LQFP100_PIN_33 -> unconnected-(J_CARDX_L_1-Pad45)
- J_CARDX_L_1 pad 46: unconnected-(J_CARDX_L_1-Pad46) -> /Profile_Switching/LQFP100_PIN_14
- J_CARDX_L_1 pad 47: /Profile_Switching/LQFP100_PIN_34 -> unconnected-(J_CARDX_L_1-Pad47)
- J_CARDX_L_1 pad 52: unconnected-(J_CARDX_L_1-Pad52) -> /Profile_Switching/LQFP100_PIN_68
- J_CARDX_L_1 pad 53: /Profile_Switching/LQFP64_PIN_42 -> unconnected-(J_CARDX_L_1-Pad53)
- J_CARDX_L_1 pad 55: /Profile_Switching/LQFP64_PIN_43 -> unconnected-(J_CARDX_L_1-Pad55)
- J_CARDX_L_1 pad 61: unconnected-(J_CARDX_L_1-Pad61) -> /Profile_Switching/LQFP100_PIN_10
- J_CARDX_L_1 pad 64: unconnected-(J_CARDX_L_1-Pad64) -> /Profile_Switching/LQFP64_PIN_47
- J_CARDX_L_1 pad 72: /Profile_Switching/LQFP100_PIN_19 -> unconnected-(J_CARDX_L_1-Pad72)
- J_CARDX_L_1 pad 73: /Profile_Switching/LQFP64_PIN_60 -> /Profile_Switching/LQFP100_PIN_19
- J_CARDX_L_1 pad 75: /Profile_Switching/LQFP64_PIN_60 -> unconnected-(J_CARDX_L_1-Pad75)
- J_CARDX_L_1 pad 77: unconnected-(J_CARDX_L_1-Pad77) -> /Profile_Switching/LQFP64_PIN_33
- J_CARDX_L_1 pad 79: /Profile_Switching/LQFP100_PIN_14 -> /Profile_Switching/LQFP64_PIN_17
- J_CARDX_L_1 pad 81: /Profile_Switching/LQFP100_PIN_94 -> unconnected-(J_CARDX_L_1-Pad81)
- J_CARDX_L_1 pad 84: /Profile_Switching/LQFP64_PIN_33 -> unconnected-(J_CARDX_L_1-Pad84)
- J_CARDX_L_1 pad 86: unconnected-(J_CARDX_L_1-Pad86) -> TARGET_POWER_SUPPLY
- J_CARDX_L_1 pad 87: unconnected-(J_CARDX_L_1-Pad87) -> TARGET_POWER_SUPPLY
- J_CARDX_L_1 pad 88: unconnected-(J_CARDX_L_1-Pad88) -> TARGET_POWER_SUPPLY
- J_CARDX_L_1 pad 90: /Profile_Switching/LQFP64_PIN_17 -> TARGET_POWER_SUPPLY
- J_CARDX_L_1 pad 91: unconnected-(J_CARDX_L_1-Pad91) -> TARGET_POWER_SUPPLY
- J_CARDX_L_1 pad 92: unconnected-(J_CARDX_L_1-Pad92) -> TARGET_POWER_SUPPLY
- J_CARDX_L_1 pad 95: unconnected-(J_CARDX_L_1-Pad95) -> TARGET_POWER_SUPPLY
- J_CARDX_L_1 pad 96: TARGET_POWER_SUPPLY -> unconnected-(J_CARDX_L_1-Pad96)
- J_CARDX_L_1 pad 99: unconnected-(J_CARDX_L_1-Pad99) -> TARGET_POWER_SUPPLY
- LS3 pad 4: /Profile_Switching/LQFP100_PIN_34 -> /Profile_Switching/LQFP100_PIN_69
- LS3 pad 5: /Profile_Switching/LQFP100_PIN_33 -> /Profile_Switching/LQFP100_PIN_68
- R41 pad 1: Net-(3.3V_EN1-Pad3) -> 3V3
- R41 pad 2: 3V3 -> Net-(3.3V_EN1-Pad3)
- R62 pad 1: Net-(STM32H1-PC11) -> 3V3
- R62 pad 2: MCU_1V8_FLAG -> Net-(DEC1-G1)
- R63 pad 1: Net-(D6-K) -> Net-(STM32H1-PA3)
- R63 pad 2: USART2_TX -> MCU_3V3_FLAG
- STM32H1 pad 10: unconnected-(STM32H1-PF0-Pad10) -> CARD_ID0_N
- STM32H1 pad 111: MCU_TARGET_PROFILE_ENABLE -> unconnected-(STM32H1-PC10-Pad111)
- STM32H1 pad 112: Net-(STM32H1-PC11) -> 3V3_ENABLE
- STM32H1 pad 113: Net-(STM32H1-PC12) -> unconnected-(STM32H1-PC12-Pad113)
- STM32H1 pad 125: unconnected-(STM32H1-PG10-Pad125) -> TARGET_PWR_ENABLE
- STM32H1 pad 133: /Parent_MCU/LCD_DATA/COMMAND -> unconnected-(STM32H1-PB3-Pad133)
- STM32H1 pad 134: /Parent_MCU/LCD_NRST -> unconnected-(STM32H1-PB4-Pad134)
- STM32H1 pad 136: unconnected-(STM32H1-PB6-Pad136) -> MCU_TARGET_PROFILE_ENABLE
- STM32H1 pad 18: LQFP64_ENABLE -> unconnected-(STM32H1-PF6-Pad18)
- STM32H1 pad 19: LQFP100_ENABLE -> unconnected-(STM32H1-PF7-Pad19)
- STM32H1 pad 36: Net-(D6-K) -> Net-(STM32H1-PA2)
- STM32H1 pad 37: Net-(D7-K) -> Net-(STM32H1-PA3)
- STM32H1 pad 57: unconnected-(STM32H1-PG1-Pad57) -> /Parent_MCU/LCD_DATA/COMMAND
- STM32H1 pad 58: unconnected-(STM32H1-PE7-Pad58) -> /Parent_MCU/LCD_NRST
- STM32H1 pad 64: unconnected-(STM32H1-PE11-Pad64) -> MCU_PROFILE_SEL1
- STM32H1 pad 65: unconnected-(STM32H1-PE12-Pad65) -> MCU_PROFILE_SEL2
- STM32H1 pad 66: unconnected-(STM32H1-PE13-Pad66) -> MCU_PROFILE_SEL3
- STM32H1 pad 7: 1V8_ENABLE -> unconnected-(STM32H1-PC13-Pad7)
- STM32H1 pad 75: unconnected-(STM32H1-PB14-Pad75) -> LQFP100_ENABLE
- STM32H1 pad 79: unconnected-(STM32H1-PD10-Pad79) -> LQFP64_ENABLE
- STM32H1 pad 8: 3V3_ENABLE -> CARD_ID2_N
- STM32H1 pad 80: unconnected-(STM32H1-PD11-Pad80) -> 1V8_ENABLE
- STM32H1 pad 9: unconnected-(STM32H1-PC15-Pad9) -> CARD_ID1_N
- STM32H1 pad 90: CARD_ID0_N -> unconnected-(STM32H1-PG5-Pad90)
- STM32H1 pad 91: CARD_ID1_N -> unconnected-(STM32H1-PG6-Pad91)
- STM32H1 pad 92: CARD_ID2_N -> unconnected-(STM32H1-PG7-Pad92)
- STM32H1 pad 97: MCU_PROFILE_SEL1 -> unconnected-(STM32H1-PC7-Pad97)
- STM32H1 pad 98: MCU_PROFILE_SEL2 -> unconnected-(STM32H1-PC8-Pad98)
- STM32H1 pad 99: MCU_PROFILE_SEL3 -> unconnected-(STM32H1-PC9-Pad99)
Routing:
- net GND: track 139.4 -> 15.0 mm, vias 125 -> 35
- net TARGET_POWER_SUPPLY: track 3.05 -> 125.2 mm, vias 0 -> 2
- net TARGET_PROFILE_4: track 0.00 -> 116.9 mm, vias 0 -> 2
- net LQFP100_ENABLE: track 0.00 -> 112.1 mm, vias 0 -> 3
- net 3V3_ENABLE: track 0.00 -> 101.6 mm, vias 0 -> 4
- net LQFP64_ENABLE: track 0.00 -> 95.9 mm, vias 0 -> 4
- net 1V8_ENABLE: track 3.25 -> 91.2 mm, vias 0 -> 5
- net CARD_ID0_N: track 0.00 -> 86.2 mm, vias 0 -> 2
- net CARD_ID1_N: track 0.00 -> 82.9 mm, vias 0 -> 2
- net CARD_ID2_N: track 0.00 -> 82.8 mm, vias 0 -> 2
- net /Profile_Switching/LQFP100_PIN_68: track 0.00 -> 81.9 mm, vias 0 -> 3
- net /Profile_Switching/LQFP100_PIN_94: track 0.00 -> 80.4 mm, vias 0 -> 3
- net /Profile_Switching/LQFP100_PIN_14: track 0.00 -> 76.2 mm, vias 0 -> 2
- net /Profile_Switching/LQFP64_PIN_43: track 0.00 -> 66.7 mm, vias 0 -> 3
- net MCU_PROFILE_SEL1: track 0.00 -> 65.3 mm, vias 0 -> 2
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- removed copper zone on F.Cu, net 5V
- removed copper zone on F.Cu, net Net-(EFUSE1-ITIMER)
Other:
- board text added: "DEBUG"
- board text added: "Delete vias - GND Fill"
- board text added: "Fix this area"
- board text added: "MOVE LCD SCREEN - ADD MECHANICAL SPACERS"
- board text added: "Orthogonal pad exits, keep traces nice"
- board text added: "R3"

Commit message: Finished Parent board
Parts:
- moved 1V8_EN1 4.23 mm to (42.5, 130.0)
- moved 3.3V_EN1 4.23 mm to (42.8, 142.3)
- moved C50 4.23 mm to (41.1, 121.9)
- moved R39 4.23 mm to (48.6, 139.0)
- moved R41 4.23 mm to (48.4, 145.6)
- moved R42 4.23 mm to (48.4, 133.3)
- moved R52 4.23 mm to (41.2, 120.4)
- moved R53 4.23 mm to (44.9, 121.1)
- moved R63 4.23 mm to (49.5, 142.3)
- moved R81 4.23 mm to (49.0, 130.0)
- moved R40 4.23 mm to (48.7, 126.7)
- moved RESET1 4.23 mm to (42.6, 114.3)
- moved C82 2.33 mm to (87.2, 53.6)
- moved C8 0.35 mm to (48.3, 68.8)
- moved C68 0.10 mm to (57.4, 95.2)
Routing:
- net 3V3: track 152.6 -> 165.2 mm, vias 60 -> 67
- net unconnected-(STM32H1-PD5-Pad119): track 2.75 -> 0.00 mm
- net Net-(STM32H1-PA3): track 47.0 -> 49.7 mm
- net GND: track 15.0 -> 12.8 mm, vias 35 -> 221
- net Net-(STM32H1-NRST): track 26.5 -> 28.2 mm
- net Net-(STM32H1-PA2): track 33.9 -> 35.6 mm
- added copper zone on B.Cu, net GND
Other:
- board text removed: "1V8_EN"
- board text removed: "3V3"
- board text removed: "3V3_EN"
- board text removed: "BOTH FOR AUTO"
- board text removed: "CS"
- board text removed: "D/C"
- board text removed: "Delete vias - GND Fill"
- board text removed: "Fix this area"
- board text removed: "GND"
- board text removed: "LITE"
- board text removed: "MISO"
- board text removed: "MOSI"
- board text removed: "MOVE LCD SCREEN - ADD MECHANICAL SPACERS"
- board text removed: "NSS"
- board text removed: "Orthogonal pad exits, keep traces nice"
- board text removed: "RESET"
- board text removed: "SCK"
- board text removed: "SWDCLK"
- board text removed: "SWDIO"
- board text removed: "TARGET POWER SEL"

Commit message: sockets
fdsfd
Changed lines of the file:
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@@
 		(tags "test point SMD pad rectangle square")
 		(property "Reference" "3V1"
-			(at 0 -1.448 0)
+			(at 0 1.7625 0)
 			(layer "F.SilkS")
 			(effects
@@
 		(tags "capacitor")
 		(property "Reference" "C36"
-			(at 0 -1.85 90)
+			(at 0 -2.85 90)
 			(layer "F.SilkS")
 			(effects
@@
 		(tags "resistor")
 		(property "Reference" "R74"
-			(at 0 -1.43 0)
+			(at 0 -1.63 0)
 			(layer "F.SilkS")
 			(effects
