File: CG Files.kicad_pcb (KiCad board)
At the start: 4 copper layers, 354 parts, among them J1 Conn_01x16_Pin, J10 Conn_01x16_Pin, J11 Conn_01x16_Pin, J12 Conn_01x16_Pin, J13 Conn_01x25_Pin, J14 Conn_01x25_Pin, J15 Conn_01x25_Pin, J16 Conn_01x25_Pin, J2 Conn_01x16_Pin, J3 Conn_01x16_Pin, J4 Conn_01x16_Pin, J5 Conn_01x25_Pin, J6 Conn_01x25_Pin, J7 Conn_01x25_Pin, J8 Conn_01x25_Pin, J9 Conn_01x16_Pin, Y1 Crystal_GND24

Commit message: xzcxzc
Parts:
- removed J_SOCKET_100_2: IC51-1004-809, MyFootprints:YAMAICHI_IC51-1004-809
- removed J_SOCKET_64_2: IC51-0644-807, MyFootprints:YAMAICHI_IC51-0644-807
- LQFP100_DATA_1, LQFP100_DEAD_1, LQFP64_DATA_1, LQFP64_DEAD_1: moved to B.Cu
- moved PARENT_DEAD1 235.3 mm to (196.3, 53.4), turned to -90 degrees
- moved J3 224.3 mm to (239.6, 34.1), turned to 0 degrees
- moved J4 219.5 mm to (235.5, 34.1), turned to 0 degrees
- moved J1 209.6 mm to (303.6, 72.4), turned to 180 degrees
- moved J2 207.1 mm to (308.1, 72.3), turned to 180 degrees
- moved LQFP64_DATA_1 194.2 mm to (314.8, 52.9), turned to -90 degrees
- moved LQFP64_DEAD_1 194.0 mm to (226.9, 53.4), turned to -90 degrees
- moved C148 174.4 mm to (558.3, 288.3)
- moved C127 174.4 mm to (546.3, 288.3)
- moved C134 174.4 mm to (550.3, 288.3)
- moved C141 174.4 mm to (554.3, 288.3)
- moved C144 174.4 mm to (558.3, 278.2)
- moved C145 174.4 mm to (558.3, 280.8)
- moved C146 174.4 mm to (558.3, 283.3)
- moved C147 174.4 mm to (558.3, 285.8)
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Routing:
- net /Profile_Switching/64_1: track 0.00 -> 1.32 mm
