File: CG Files.kicad_pcb (KiCad board)
At the start: 4 copper layers, 325.2 x 167.6 mm, 323 parts, among them J1 Conn_01x16_Pin, J10 Conn_01x08_Pin, J11 Conn_01x09_Pin, J12 Conn_01x08_Pin, J13 Conn_01x08_Pin, J14 Conn_01x09_Pin, J15 Conn_01x08_Pin, J16 Conn_01x08_Pin, J2 Conn_01x16_Pin, J3 Conn_01x16_Pin, J4 Conn_01x16_Pin, J5 Conn_01x08_Pin, J6 Conn_01x09_Pin, J7 Conn_01x08_Pin, J8 Conn_01x09_Pin, J9 Conn_01x08_Pin, Y1 Crystal_GND24

Commit message: silkscreen
fdsfsd
Parts:
- moved R54 1.86 mm to (51.5, 80.8)
- moved BOOT0_LED 0.67 mm to (51.4, 83.7)
- moved C90 0.37 mm to (87.8, 98.2)
- moved C77 0.10 mm to (85.6, 69.7)
- renumbered BOOT0_LED1 to BOOT0_LED
Routing:
- net GND: track 51.7 -> 77.3 mm, vias 280 -> 277
- net 3V3: track 198.6 -> 202.3 mm, vias 72 -> 70
- net Net-(STM32H1-BOOT0): track 18.4 -> 20.1 mm
- net Net-(BOOT0_LED1-A): track 15.8 -> 17.2 mm
- net TARGET_BOOT0_CONTROL: track 51.4 -> 50.6 mm
- net Net-(LS2-OE): track 11.5 -> 12.2 mm
- net Net-(INV6-Pad4): track 2.67 -> 3.26 mm
Other:
- board size 325.2 x 167.6 mm -> 427.4 x 168.3 mm
