File: Plug_in_Cards.kicad_sch (KiCad schematic)
At the start: 0 parts

Commit message: target routing
d fsdf dsfd
Parts:
- added C123, C124, C125, C126, C127, C128, C129, C130, C131, C132, C133, C134, C135, C136, C137, C138, C139, C140, C141, C142, C143, C144, C145, C146, C147, C148, C149: 2.2u, Capacitor_SMD:C_0603_1608Metric, symbol Device:C_Small_US
- added J10, J11, J12, J9: Conn_01x16_Pin, Connector_PinHeader_2.54mm:PinHeader_1x16_P2.54mm_Vertical, symbol Connector:Conn_01x16_Pin
- added J13, J14, J15, J16: Conn_01x25_Pin, Connector_PinHeader_2.54mm:PinHeader_1x25_P2.54mm_Vertical, symbol Connector:Conn_01x25_Pin
- added J_SOCKET_100_2: IC51-1004-809, MyFootprints:YAMAICHI_IC51-1004-809, symbol MySymbols:IC51-1004-809
- added J_SOCKET_64_2: IC51-0644-807, MyFootprints:YAMAICHI_IC51-0644-807, symbol MySymbols:IC51-0644-807
Connections:
- new net 100_1: J13.1 (Pin_1), J_SOCKET_100_2.1
- new net 100_10: J14.5 (Pin_5), J_SOCKET_100_2.10
- new net 100_100: C148.1, J16.25 (Pin_25), J_SOCKET_100_2.100
- new net 100_11: C139.1, J13.6 (Pin_6), J_SOCKET_100_2.11
- new net 100_12: J14.6 (Pin_6), J_SOCKET_100_2.12
- new net 100_13: J13.7 (Pin_7), J_SOCKET_100_2.13
- new net 100_14: J14.7 (Pin_7), J_SOCKET_100_2.14
- new net 100_15: J13.8 (Pin_8), J_SOCKET_100_2.15
- new net 100_16: J14.8 (Pin_8), J_SOCKET_100_2.16
- new net 100_17: J13.9 (Pin_9), J_SOCKET_100_2.17
- new net 100_18: J14.9 (Pin_9), J_SOCKET_100_2.18
- new net 100_19: C143.1, J13.10 (Pin_10), J_SOCKET_100_2.19
- new net 100_2: J14.1 (Pin_1), J_SOCKET_100_2.2
- new net 100_20: J14.10 (Pin_10), J_SOCKET_100_2.20
- new net 100_21: C137.1, J13.11 (Pin_11), J_SOCKET_100_2.21
- new net 100_22: C135.1, J14.11 (Pin_11), J_SOCKET_100_2.22
- new net 100_23: J13.12 (Pin_12), J_SOCKET_100_2.23
- new net 100_24: J14.12 (Pin_12), J_SOCKET_100_2.24
- new net 100_25: J13.13 (Pin_13), J_SOCKET_100_2.25
- new net 100_26: J14.13 (Pin_13), J_SOCKET_100_2.26
- new net 100_27: J13.14 (Pin_14), J_SOCKET_100_2.27
- new net 100_28: C140.1, J14.14 (Pin_14), J_SOCKET_100_2.28
- new net 100_29: J13.15 (Pin_15), J_SOCKET_100_2.29
- new net 100_3: J13.2 (Pin_2), J_SOCKET_100_2.3
- new net 100_30: J14.15 (Pin_15), J_SOCKET_100_2.30
- new net 100_31: J13.16 (Pin_16), J_SOCKET_100_2.31
- new net 100_32: J14.16 (Pin_16), J_SOCKET_100_2.32
- new net 100_33: J13.17 (Pin_17), J_SOCKET_100_2.33
- new net 100_34: J14.17 (Pin_17), J_SOCKET_100_2.34
- new net 100_35: J13.18 (Pin_18), J_SOCKET_100_2.35
- new net 100_36: J14.18 (Pin_18), J_SOCKET_100_2.36
- new net 100_37: J13.19 (Pin_19), J_SOCKET_100_2.37
- new net 100_38: J14.19 (Pin_19), J_SOCKET_100_2.38
- new net 100_39: J13.20 (Pin_20), J_SOCKET_100_2.39
- new net 100_4: J14.2 (Pin_2), J_SOCKET_100_2.4
- new net 100_40: J14.20 (Pin_20), J_SOCKET_100_2.40
- new net 100_41: J13.21 (Pin_21), J_SOCKET_100_2.41
- new net 100_42: J14.21 (Pin_21), J_SOCKET_100_2.42
- new net 100_43: C141.1, J13.22 (Pin_22), J_SOCKET_100_2.43
- new net 100_44: J14.22 (Pin_22), J_SOCKET_100_2.44
- new net 100_45: J13.23 (Pin_23), J_SOCKET_100_2.45
- new net 100_46: J14.23 (Pin_23), J_SOCKET_100_2.46
- new net 100_47: J13.24 (Pin_24), J_SOCKET_100_2.47
- new net 100_48: C136.1, J14.24 (Pin_24), J_SOCKET_100_2.48
- new net 100_49: C134.1, J13.25 (Pin_25), J_SOCKET_100_2.49
- new net 100_5: J13.3 (Pin_3), J_SOCKET_100_2.5
- new net 100_50: C142.1, J14.25 (Pin_25), J_SOCKET_100_2.50
- new net 100_51: J15.1 (Pin_1), J_SOCKET_100_2.51
- new net 100_52: J16.1 (Pin_1), J_SOCKET_100_2.52
- new net 100_53: J15.2 (Pin_2), J_SOCKET_100_2.53
- new net 100_54: J16.2 (Pin_2), J_SOCKET_100_2.54
- new net 100_55: J15.3 (Pin_3), J_SOCKET_100_2.55
- new net 100_56: C144.1, J16.3 (Pin_3), J_SOCKET_100_2.56
- new net 100_57: J15.4 (Pin_4), J_SOCKET_100_2.57
- new net 100_58: J16.4 (Pin_4), J_SOCKET_100_2.58
- new net 100_59: J15.5 (Pin_5), J_SOCKET_100_2.59
- new net 100_6: C138.1, J14.3 (Pin_3), J_SOCKET_100_2.6
- new net 100_60: J16.5 (Pin_5), J_SOCKET_100_2.60
- new net 100_61: J15.6 (Pin_6), J_SOCKET_100_2.61
- new net 100_62: C145.1, J16.6 (Pin_6), J_SOCKET_100_2.62
- new net 100_63: J15.7 (Pin_7), J_SOCKET_100_2.63
- new net 100_64: J16.7 (Pin_7), J_SOCKET_100_2.64
- new net 100_65: J15.8 (Pin_8), J_SOCKET_100_2.65
- new net 100_66: J16.8 (Pin_8), J_SOCKET_100_2.66
- new net 100_67: J15.9 (Pin_9), J_SOCKET_100_2.67
- new net 100_68: J16.9 (Pin_9), J_SOCKET_100_2.68
- new net 100_69: J15.10 (Pin_10), J_SOCKET_100_2.69
- new net 100_7: J13.4 (Pin_4), J_SOCKET_100_2.7
- new net 100_70: J16.10 (Pin_10), J_SOCKET_100_2.70
- new net 100_71: J15.11 (Pin_11), J_SOCKET_100_2.71
- new net 100_72: J16.11 (Pin_11), J_SOCKET_100_2.72
- new net 100_73: C146.1, J15.12 (Pin_12), J_SOCKET_100_2.73
- new net 100_74: J16.12 (Pin_12), J_SOCKET_100_2.74
- new net 100_75: C147.1, J15.13 (Pin_13), J_SOCKET_100_2.75
- new net 100_76: C149.1, J16.13 (Pin_13), J_SOCKET_100_2.76
- new net 100_77: J15.14 (Pin_14), J_SOCKET_100_2.77
- new net 100_78: J16.14 (Pin_14), J_SOCKET_100_2.78
- new net 100_79: J15.15 (Pin_15), J_SOCKET_100_2.79
- new net 100_8: J14.4 (Pin_4), J_SOCKET_100_2.8
- new net 100_80: J16.15 (Pin_15), J_SOCKET_100_2.80
- new net 100_81: J15.16 (Pin_16), J_SOCKET_100_2.81
- new net 100_82: J16.16 (Pin_16), J_SOCKET_100_2.82
- new net 100_83: J15.17 (Pin_17), J_SOCKET_100_2.83
- new net 100_84: J16.17 (Pin_17), J_SOCKET_100_2.84
- new net 100_85: J15.18 (Pin_18), J_SOCKET_100_2.85
- new net 100_86: J16.18 (Pin_18), J_SOCKET_100_2.86
- new net 100_87: J15.19 (Pin_19), J_SOCKET_100_2.87
- new net 100_88: J16.19 (Pin_19), J_SOCKET_100_2.88
- new net 100_89: J15.20 (Pin_20), J_SOCKET_100_2.89
- new net 100_9: J13.5 (Pin_5), J_SOCKET_100_2.9
- new net 100_90: J16.20 (Pin_20), J_SOCKET_100_2.90
- new net 100_91: J15.21 (Pin_21), J_SOCKET_100_2.91
- new net 100_92: J16.21 (Pin_21), J_SOCKET_100_2.92
- new net 100_93: J15.22 (Pin_22), J_SOCKET_100_2.93
- new net 100_94: J16.22 (Pin_22), J_SOCKET_100_2.94
- new net 100_95: J15.23 (Pin_23), J_SOCKET_100_2.95
- new net 100_96: J16.23 (Pin_23), J_SOCKET_100_2.96
- new net 100_97: J15.24 (Pin_24), J_SOCKET_100_2.97
- new net 100_98: J16.24 (Pin_24), J_SOCKET_100_2.98
- new net 100_99: J15.25 (Pin_25), J_SOCKET_100_2.99
- new net 64_1: C126.1, J9.1 (Pin_1), J_SOCKET_64_2.1
- new net 64_10: J10.5 (Pin_5), J_SOCKET_64_2.10
- new net 64_11: J9.6 (Pin_6), J_SOCKET_64_2.11
- new net 64_12: J10.6 (Pin_6), J_SOCKET_64_2.12
- new net 64_13: C127.1, J9.7 (Pin_7), J_SOCKET_64_2.13
- new net 64_14: J10.7 (Pin_7), J_SOCKET_64_2.14
- new net 64_15: J9.8 (Pin_8), J_SOCKET_64_2.15
- new net 64_16: J10.8 (Pin_8), J_SOCKET_64_2.16
- new net 64_17: C128.1, J9.9 (Pin_9), J_SOCKET_64_2.17
- new net 64_18: J10.9 (Pin_9), J_SOCKET_64_2.18
- new net 64_19: C125.1, J9.10 (Pin_10), J_SOCKET_64_2.19
- new net 64_2: J10.1 (Pin_1), J_SOCKET_64_2.2
- new net 64_20: J10.10 (Pin_10), J_SOCKET_64_2.20
- new net 64_21: J9.11 (Pin_11), J_SOCKET_64_2.21
- new net 64_22: J10.11 (Pin_11), J_SOCKET_64_2.22
- new net 64_23: J9.12 (Pin_12), J_SOCKET_64_2.23
- new net 64_24: J10.12 (Pin_12), J_SOCKET_64_2.24
- new net 64_25: J9.13 (Pin_13), J_SOCKET_64_2.25
- new net 64_26: J10.13 (Pin_13), J_SOCKET_64_2.26
- new net 64_27: J9.14 (Pin_14), J_SOCKET_64_2.27
- new net 64_28: J10.14 (Pin_14), J_SOCKET_64_2.28
- new net 64_29: J9.15 (Pin_15), J_SOCKET_64_2.29
- new net 64_3: J9.2 (Pin_2), J_SOCKET_64_2.3
- new net 64_30: C129.1, J10.15 (Pin_15), J_SOCKET_64_2.30
- new net 64_31: C124.1, J9.16 (Pin_16), J_SOCKET_64_2.31
- new net 64_32: C123.1, J10.16 (Pin_16), J_SOCKET_64_2.32
- new net 64_33: C130.1, J11.1 (Pin_1), J_SOCKET_64_2.33
- new net 64_34: J12.1 (Pin_1), J_SOCKET_64_2.34
- new net 64_35: J11.2 (Pin_2), J_SOCKET_64_2.35
- new net 64_36: J12.2 (Pin_2), J_SOCKET_64_2.36
- new net 64_37: J11.3 (Pin_3), J_SOCKET_64_2.37
- new net 64_38: J12.3 (Pin_3), J_SOCKET_64_2.38
- new net 64_39: J11.4 (Pin_4), J_SOCKET_64_2.39
- new net 64_4: J10.2 (Pin_2), J_SOCKET_64_2.4
- new net 64_40: J12.4 (Pin_4), J_SOCKET_64_2.40
- new net 64_41: J11.5 (Pin_5), J_SOCKET_64_2.41
- new net 64_42: J12.5 (Pin_5), J_SOCKET_64_2.42
- new net 64_43: J11.6 (Pin_6), J_SOCKET_64_2.43
- new net 64_44: J12.6 (Pin_6), J_SOCKET_64_2.44
- new net 64_45: J11.7 (Pin_7), J_SOCKET_64_2.45
- new net 64_46: J12.7 (Pin_7), J_SOCKET_64_2.46
- new net 64_47: C133.1, J11.8 (Pin_8), J_SOCKET_64_2.47
- new net 64_48: C131.2, J12.8 (Pin_8), J_SOCKET_64_2.48
- new net 64_49: J11.9 (Pin_9), J_SOCKET_64_2.49
- new net 64_5: J9.3 (Pin_3), J_SOCKET_64_2.5
- new net 64_50: J12.9 (Pin_9), J_SOCKET_64_2.50
- new net 64_51: J11.10 (Pin_10), J_SOCKET_64_2.51
- new net 64_52: J12.10 (Pin_10), J_SOCKET_64_2.52
- new net 64_53: J11.11 (Pin_11), J_SOCKET_64_2.53
- new net 64_54: J12.11 (Pin_11), J_SOCKET_64_2.54
- new net 64_55: J11.12 (Pin_12), J_SOCKET_64_2.55
- new net 64_56: J12.12 (Pin_12), J_SOCKET_64_2.56
- new net 64_57: J11.13 (Pin_13), J_SOCKET_64_2.57
- new net 64_58: J12.13 (Pin_13), J_SOCKET_64_2.58
- new net 64_59: J11.14 (Pin_14), J_SOCKET_64_2.59
- new net 64_6: J10.3 (Pin_3), J_SOCKET_64_2.6
- new net 64_60: J12.14 (Pin_14), J_SOCKET_64_2.60
- new net 64_61: J11.15 (Pin_15), J_SOCKET_64_2.61
- new net 64_62: J12.15 (Pin_15), J_SOCKET_64_2.62
- new net 64_63: J11.16 (Pin_16), J_SOCKET_64_2.63
- new net 64_64: C132.1, J12.16 (Pin_16), J_SOCKET_64_2.64
- new net 64_7: J9.4 (Pin_4), J_SOCKET_64_2.7
- new net 64_8: J10.4 (Pin_4), J_SOCKET_64_2.8
- new net 64_9: J9.5 (Pin_5), J_SOCKET_64_2.9
- new net GND: C123.2, C124.2, C125.2, C126.2, C127.2, C128.2, C129.2, C130.2, C131.1, C132.2, C133.2, C134.2, C135.2, C136.2, C137.2, C138.2, C139.2, C140.2, C141.2, C142.2, C143.2, C144.2, C145.2, C146.2, C147.2, C148.2, C149.2

Commit message: xzcxzc
Parts:
- removed C123, C124, C125, C126, C127, C128, C129, C130, C131, C132, C133, C134, C135, C136, C137, C138, C139, C140, C141, C142, C143, C144, C145, C146, C147, C148, C149: 2.2u, Capacitor_SMD:C_0603_1608Metric, symbol Device:C_Small_US
- removed J10, J11, J12, J9: Conn_01x16_Pin, Connector_PinHeader_2.54mm:PinHeader_1x16_P2.54mm_Vertical, symbol Connector:Conn_01x16_Pin
- removed J13, J14, J15, J16: Conn_01x25_Pin, Connector_PinHeader_2.54mm:PinHeader_1x25_P2.54mm_Vertical, symbol Connector:Conn_01x25_Pin
- removed J_SOCKET_100_2: IC51-1004-809, MyFootprints:YAMAICHI_IC51-1004-809, symbol MySymbols:IC51-1004-809
- removed J_SOCKET_64_2: IC51-0644-807, MyFootprints:YAMAICHI_IC51-0644-807, symbol MySymbols:IC51-0644-807
