File: Profile_Switching.kicad_sch (KiCad schematic)
At the start: 110 parts

Commit message: finished routing
//TODO
-> add mechanical support
-> daughter board
-> recheck nodes/conections
-> silk screen
Parts:
- removed BUF7, BUF9: 74AHC1G125, Package_TO_SOT_SMD:SOT-553, symbol 74xGxx:74AHC1G125
- removed C101, C102, C103, C106, C108, C111, C112, C88, C90, C91, C93, C94, C95, C96, C97, C98, C99: .1uF, Capacitor_SMD:C_0402_1005Metric, symbol Device:C_Small_US
- removed INV7: 74LVC1GU04DRLR, Package_TO_SOT_SMD:SOT-553, symbol 74xGxx:74LVC1GU04DRL
- removed LS2: TXS0102DCUR, Package_SO:VSSOP-8_2.3x2mm_P0.5mm, symbol Logic_LevelTranslator:TXS0102DCU
- removed R83: 10k, Resistor_SMD:R_0603_1608Metric, symbol Device:R
- removed R84: 12k, Resistor_SMD:R_0603_1608Metric, symbol Device:R
- added R62: 10k, Resistor_SMD:R_0603_1608Metric, symbol Device:R
- renumbered C89 to C88, C92 to C89, C100 to C92, C104 to C94, C105 to C95, C107 to C96, C109 to C97, C110 to C98, R66 to R64, R67 to R65, R68 to R66, R69 to R67, R70 to R68, R71 to R69, R72 to R70, R73 to R71, R74 to R72, R75 to R73, R76 to R74, R77 to R75, R78 to R76, R79 to R77, R80 to R78, R81 to R79, R82 to R80, R85 to R83, R86 to R84, R87 to R85, R88 to R86, R89 to R87, R90 to R88, R91 to R89, R92 to R90, R93 to R91
Connections:
- net 3V3: now also R62.1
- net LQFP100_ENABLE: now also J_CARDX_L_1.03; no longer J_CARDX_L_1.27
- net LQFP100_PIN_10: now also J_CARDX_L_1.61; no longer J_CARDX_L_1.12
- net LQFP100_PIN_14: now also J_CARDX_L_1.46; no longer J_CARDX_L_1.79
- net LQFP100_PIN_19: now also J_CARDX_L_1.73; no longer J_CARDX_L_1.72
- net LQFP100_PIN_22: now also J_CARDX_L_1.118; no longer J_CARDX_L_1.113
- net LQFP100_PIN_27: now also J_CARDX_L_1.08; no longer J_CARDX_L_1.18
- net LQFP100_PIN_68: now also BUF13.2, J_CARDX_L_1.52, LS3.5 (A1); no longer J_CARDX_L_1.35
- net LQFP100_PIN_69: now also BUF11.4, J_CARDX_L_1.115, LS3.4 (A2); no longer J_CARDX_L_1.37
- net LQFP100_PIN_94: now also J_CARDX_L_1.40; no longer J_CARDX_L_1.81
- net LQFP64_ENABLE: now also J_CARDX_L_1.05; no longer J_CARDX_L_1.25
- net LQFP64_PIN_17: now also J_CARDX_L_1.79; no longer J_CARDX_L_1.90
- net LQFP64_PIN_19: now also J_CARDX_L_1.109; no longer J_CARDX_L_1.114
- net LQFP64_PIN_33: now also J_CARDX_L_1.77; no longer J_CARDX_L_1.84
- net LQFP64_PIN_42: now also J_CARDX_L_1.117; no longer J_CARDX_L_1.53
- net LQFP64_PIN_43: now also J_CARDX_L_1.37; no longer J_CARDX_L_1.55
- net LQFP64_PIN_47: now also J_CARDX_L_1.64; no longer J_CARDX_L_1.01
- net LQFP64_PIN_48: now also J_CARDX_L_1.113; no longer J_CARDX_L_1.119
- net LQFP64_PIN_60: now also J_CARDX_L_1.120; no longer J_CARDX_L_1.73, J_CARDX_L_1.75
- net LQFP64_PIN_7: now also J_CARDX_L_1.119
- net TARGET_POWER_SUPPLY: now also J_CARDX_L_1.86, J_CARDX_L_1.87, J_CARDX_L_1.88, J_CARDX_L_1.90, J_CARDX_L_1.91, J_CARDX_L_1.92, J_CARDX_L_1.95, J_CARDX_L_1.99; no longer J_CARDX_L_1.07, J_CARDX_L_1.101, J_CARDX_L_1.102, J_CARDX_L_1.105, J_CARDX_L_1.108, J_CARDX_L_1.109, J_CARDX_L_1.120, J_CARDX_L_1.96
- removed net LQFP100_PIN_33: BUF13.2, J_CARDX_L_1.45, LS3.5 (A1)
- removed net LQFP100_PIN_34: BUF11.4, J_CARDX_L_1.47, LS3.4 (A2)
- net MCU_TARGET_PROFILE_ENABLE: no longer names the net of DEC1.6 (G1)
- net MCU_TARGET_PROFILE_ENABLE: now also R62.2
- net TARGET_PWR_ENABLE: no longer names the net of J_CARDX_L_1.02
- no-connect marks 91 -> 93
Other:
- note removed: "USART2 - 1V8"

Commit message: sockets
fdsfd
Parts:
- added DATA_1, DEAD_1, DEAD_2, J_V064CARD_L2, J_V064CARD_L3, J_V064CARD_L4: QTH-060-03-X-D-A, footprints2:SAMTEC_QTH-060-01-X-D-A, symbol MySymbols:QTH-060-03-X-D-A
- added DATA_2: QSH-060-01-X-D-A, footprints2:SAMTEC_QTH-060-01-X-D-A, symbol MySymbols:QSH-060-01-X-D-A
- added J_CARDX_L_2: QSH-060-01-X-D-A, MyFootprints:SAMTEC_QTH-060-01-X-D-A, symbol MySymbols:QSH-060-01-X-D-A
- added J_V064CARD_L1: QTH-060-03-X-D-A, footprints2:SAMTEC_QSH-060-01-X-D-A, symbol MySymbols:QTH-060-03-X-D-A
- added LQFP100_SWD1, LQFP100_USART1, LQFP64_SWD1, LQFP64_USART1: Conn_01x04_Pin, Connector_PinHeader_2.54mm:PinHeader_1x04_P2.54mm_Vertical, symbol Connector:Conn_01x04_Pin
- added PARENT_DEAD1: QSH-060-01-X-D-A, MyFootprints:SAMTEC_QSH-060-01-X-D-A, symbol MySymbols:QTH-060-03-X-D-A
- renumbered BUF12 to BUF10, BUF13 to BUF11, BUF14 to BUF12, BUF8 to BUF5, BUF5 to BUF6, BUF6 to BUF7, BUF10 to BUF8, BUF11 to BUF9, C92 to C90, C95 to C91, C96 to C92, C97 to C93, C98 to C94, C94 to C95, INV8 to INV7, LS3 to LS2, R83 to R81, R84 to R82, R85 to R83, R86 to R84, R62 to R85, R87 to R86, R88 to R87, R89 to R88, R90 to R89, R91 to R90
Connections:
- net +3V3 is gone; now on net 3V3: R88.1, R89.1, R90.1
- net 3V3: now also J_CARDX_L_2.65, J_V064CARD_L2.65
- net GND: now also DATA_1.19, DATA_1.G1 (GND1), DATA_1.G2 (GND1__1), DATA_1.G3 (GND1__2), DATA_1.G4 (GND1__3), DATA_2.23, DATA_2.G1_1 (GND1), DATA_2.G1_2 (GND1__1), DATA_2.G1_3 (GND1__2), DATA_2.G1_4 (GND1__3), J_CARDX_L_2.G2_1 (GND2), J_CARDX_L_2.G2_2 (GND2__1), J_CARDX_L_2.G2_3 (GND2__2), J_CARDX_L_2.G2_4 (GND2__3), J_V064CARD_L2.G5 (GND2), J_V064CARD_L2.G6 (GND2__1), J_V064CARD_L2.G7 (GND2__2), J_V064CARD_L2.G8 (GND2__3), LQFP100_SWD1.4 (Pin_4), LQFP100_USART1.4 (Pin_4), LQFP64_SWD1.4 (Pin_4), LQFP64_USART1.4 (Pin_4)
- new net 100_10: J_CARDX_L_2.61
- new net 100_100: J_CARDX_L_2.89
- new net 100_11: J_CARDX_L_2.78
- new net 100_14: DATA_2.46
- new net 100_19: J_CARDX_L_2.73
- new net 100_20: DATA_2.24
- new net 100_21: J_CARDX_L_2.93
- new net 100_22: J_CARDX_L_2.118
- new net 100_27: DATA_2.08
- new net 100_28: J_CARDX_L_2.95
- new net 100_49: DATA_2.30
- new net 100_50: J_CARDX_L_2.97
- new net 100_6: J_CARDX_L_2.91
- new net 100_68: DATA_2.52, LQFP100_USART1.1 (Pin_1)
- new net 100_69: J_CARDX_L_2.115, LQFP100_USART1.2 (Pin_2)
- new net 100_72: LQFP100_SWD1.1 (Pin_1)
- new net 100_74: DATA_2.36
- new net 100_75: J_CARDX_L_2.99
- new net 100_76: LQFP100_SWD1.2 (Pin_2)
- new net 100_94: DATA_2.40
- new net 100_99: DATA_2.42
- new net 64_1: J_V064CARD_L2.92
- new net 64_12: DATA_1.60
- new net 64_13: J_V064CARD_L2.86
- new net 64_17: J_V064CARD_L2.79
- new net 64_18: J_V064CARD_L2.62
- new net 64_19: J_V064CARD_L2.109
- new net 64_31: DATA_1.48
- new net 64_32: J_V064CARD_L2.88
- new net 64_33: J_V064CARD_L2.77
- new net 64_42: J_V064CARD_L2.117, LQFP64_USART1.1 (Pin_1)
- new net 64_43: DATA_1.37, LQFP64_USART1.2 (Pin_2)
- new net 64_47: J_V064CARD_L2.64
- new net 64_48: J_V064CARD_L2.113
- new net 64_60: J_V064CARD_L2.120
- new net 64_63: DATA_1.54
- new net 64_64: J_V064CARD_L2.90
- new net 64_7: J_V064CARD_L2.119
- new net SWDCLK_64: LQFP64_SWD1.2 (Pin_2)
- new net SWDIO_64: LQFP64_SWD1.1 (Pin_1)
- new net TGT_PWR: J_CARDX_L_2.87, J_V064CARD_L2.87, LQFP100_SWD1.3 (Pin_3), LQFP100_USART1.3 (Pin_3), LQFP64_SWD1.3 (Pin_3), LQFP64_USART1.3 (Pin_3)
- no-connect marks 93 -> 676
Other:
- note added: "Dead Sockets"
- note added: "LQFP100 -> dead socket"
- note added: "LQFP64 -> dead socket"
- note added: "Parent Board -> dead socket"
- note added: "TARGET BOARD DATA SOCKETS"
- note added: "UART/SWD BREAKOUT"
- note added: "target board naming - Package_pin#"
- moved on the sheet: C90, C91, C92, C93, C94, INV7, J_CARDX_L_1A, J_CARDX_L_1B, LS2, OR3, OR4, R81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

Commit message: target routing
d fsdf dsfd
Parts:
- removed DATA_1, DEAD_1, DEAD_2, J_V064CARD_L2, J_V064CARD_L3, J_V064CARD_L4: QTH-060-03-X-D-A, footprints2:SAMTEC_QTH-060-01-X-D-A, symbol MySymbols:QTH-060-03-X-D-A
- removed DATA_2: QSH-060-01-X-D-A, footprints2:SAMTEC_QTH-060-01-X-D-A, symbol MySymbols:QSH-060-01-X-D-A
- removed J_CARDX_L_2: QSH-060-01-X-D-A, MyFootprints:SAMTEC_QTH-060-01-X-D-A, symbol MySymbols:QSH-060-01-X-D-A
- added C100, C101, C103, C104, C105, C106, C108, C110, C111, C112, C113, C115, C116, C120, C121, C96, C98, C99: .1u, Capacitor_SMD:C_0402_1005Metric, symbol Device:C_Small_US
- added C102, C107, C109, C114, C117, C118, C119, C97: 2.2u, Capacitor_SMD:C_0603_1608Metric, symbol Device:C_Small_US
- added J1, J2, J3, J4: Conn_01x16_Pin, Connector_PinHeader_2.54mm:PinHeader_1x16_P2.54mm_Vertical, symbol Connector:Conn_01x16_Pin
- added J5, J6, J7, J8: Conn_01x25_Pin, Connector_PinHeader_2.54mm:PinHeader_1x25_P2.54mm_Vertical, symbol Connector:Conn_01x25_Pin
- added J_SOCKET_100_1: IC51-1004-809, MyFootprints:YAMAICHI_IC51-1004-809, symbol MySymbols:IC51-1004-809
- added J_SOCKET_64_1: IC51-0644-807, MyFootprints:YAMAICHI_IC51-0644-807, symbol MySymbols:IC51-0644-807
- added LQFP100_DATA_1, LQFP100_DEAD_1, LQFP64_DATA_1, LQFP64_DEAD_1: QTH-060-01-X-D-A, MyFootprints:SAMTEC_QTH-060-01-X-D-A, symbol MySymbols:QTH-060-01-X-D-A
- PARENT_DEAD1: footprint MyFootprints:SAMTEC_QSH-060-01-X-D-A -> footprints2:SAMTEC_QSH-060-01-X-D-A
- PARENT_DEAD1: renamed from J_V064CARD_L1; value QTH-060-03-X-D-A -> QSH-060-01-X-D-A
- renumbered BUF5 to BUF1, BUF4 to BUF10, BUF6 to BUF11, BUF7 to BUF12, BUF8 to BUF2, BUF9 to BUF3, BUF1 to BUF4, BUF10 to BUF5, BUF2 to BUF6, BUF3 to BUF7, BUF11 to BUF8, BUF12 to BUF9, C90 to C79, C79 to C80, C80 to C81, C81 to C82, C82 to C83, C83 to C84, C84 to C85, C85 to C86, C86 to C87, C91 to C88, C87 to C89, C92 to C90, C88 to C91, C93 to C92, C94 to C93, C89 to C94, INV7 to INV6, INV6 to INV7, OR3 to OR2, OR2 to OR3, R81 to R67, R67 to R68, R82 to R69, R68 to R70, R69 to R71, R70 to R72, R71 to R73, R83 to R74, R72 to R75, R73 to R76, R84 to R77, R74 to R78, R75 to R79, R76 to R80, R86 to R81, R87 to R82, R77 to R83, R78 to R84, R79 to R85, R80 to R86, R88 to R87, R89 to R88, R90 to R89, R85 to R90
Connections:
- net 100_10: now also J6.5 (Pin_5), J_SOCKET_100_1.10, LQFP100_DATA_1.61
- net 100_100: now also C121.1, J8.25 (Pin_25), J_SOCKET_100_1.100, LQFP100_DATA_1.89
- net 100_11: now also C112.1, J5.6 (Pin_6), J_SOCKET_100_1.11, LQFP100_DATA_1.78
- net 100_14: now also J6.7 (Pin_7), J_SOCKET_100_1.14, LQFP100_DATA_1.46
- net 100_19: now also C116.1, J5.10 (Pin_10), J_SOCKET_100_1.19, LQFP100_DATA_1.73
- net 100_20: now also J6.10 (Pin_10), J_SOCKET_100_1.20, LQFP100_DATA_1.24
- net 100_21: now also C110.1, J5.11 (Pin_11), J_SOCKET_100_1.21, LQFP100_DATA_1.93
- net 100_22: now also C108.1, J6.11 (Pin_11), J_SOCKET_100_1.22, LQFP100_DATA_1.118
- net 100_27: now also J5.14 (Pin_14), J_SOCKET_100_1.27, LQFP100_DATA_1.08
- net 100_28: now also C113.1, J6.14 (Pin_14), J_SOCKET_100_1.28, LQFP100_DATA_1.95
- net 100_49: now also C107.1, J5.25 (Pin_25), J_SOCKET_100_1.49, LQFP100_DATA_1.30
- net 100_50: now also C115.1, J6.25 (Pin_25), J_SOCKET_100_1.50, LQFP100_DATA_1.97
- net 100_6: now also C111.1, J6.3 (Pin_3), J_SOCKET_100_1.6, LQFP100_DATA_1.91
- net 100_68: now also J8.9 (Pin_9), J_SOCKET_100_1.68, LQFP100_DATA_1.52
- net 100_69: now also J7.10 (Pin_10), J_SOCKET_100_1.69, LQFP100_DATA_1.115
- net 100_72: now also J4.7 (Pin_7), J8.11 (Pin_11), J_SOCKET_100_1.72, J_SOCKET_64_1.46
- net 100_74: now also J8.12 (Pin_12), J_SOCKET_100_1.74, LQFP100_DATA_1.36
- net 100_75: now also C120.1, J7.13 (Pin_13), J_SOCKET_100_1.75, LQFP100_DATA_1.99
- net 100_76: now also J3.9 (Pin_9), J8.13 (Pin_13), J_SOCKET_100_1.76, J_SOCKET_64_1.49
- net 100_94: now also J8.22 (Pin_22), J_SOCKET_100_1.94, LQFP100_DATA_1.40
- net 100_99: now also J7.25 (Pin_25), J_SOCKET_100_1.99, LQFP100_DATA_1.42
- net 3V3: now also LQFP100_DATA_1.65, LQFP64_DATA_1.65
- net 64_1: now also C99.1, J1.1 (Pin_1), J_SOCKET_64_1.1, LQFP64_DATA_1.92
- net 64_12: now also J2.6 (Pin_6), J_SOCKET_64_1.12, LQFP64_DATA_1.60
- net 64_13: now also C100.1, J1.7 (Pin_7), J_SOCKET_64_1.13, LQFP64_DATA_1.86
- net 64_17: now also C101.1, J1.9 (Pin_9), J_SOCKET_64_1.17, LQFP64_DATA_1.79
- net 64_18: now also J2.9 (Pin_9), J_SOCKET_64_1.18, LQFP64_DATA_1.62
- net 64_19: now also C98.1, J1.10 (Pin_10), J_SOCKET_64_1.19, LQFP64_DATA_1.109
- net 64_31: now also C97.1, J1.16 (Pin_16), J_SOCKET_64_1.31, LQFP64_DATA_1.48
- net 64_32: now also C96.1, J2.16 (Pin_16), J_SOCKET_64_1.32, LQFP64_DATA_1.88
- net 64_33: now also C103.1, J3.1 (Pin_1), J_SOCKET_64_1.33, LQFP64_DATA_1.77
- net 64_42: now also J4.5 (Pin_5), J_SOCKET_64_1.42, LQFP64_DATA_1.117
- net 64_43: now also J3.6 (Pin_6), J_SOCKET_64_1.43, LQFP64_DATA_1.37
- net 64_47: now also C106.1, J3.8 (Pin_8), J_SOCKET_64_1.47, LQFP64_DATA_1.64
- net 64_48: now also C104.2, J4.8 (Pin_8), J_SOCKET_64_1.48, LQFP64_DATA_1.113
- net 64_60: now also J4.14 (Pin_14), J_SOCKET_64_1.60, LQFP64_DATA_1.120
- net 64_63: now also J3.16 (Pin_16), J_SOCKET_64_1.63, LQFP64_DATA_1.54
- net 64_64: now also C105.1, J4.16 (Pin_16), J_SOCKET_64_1.64, LQFP64_DATA_1.90
- net 64_7: now also J1.4 (Pin_4), J_SOCKET_64_1.7, LQFP64_DATA_1.119
- net GND: now also PARENT_DEAD1.G1 (GND1), PARENT_DEAD1.G2 (GND1__1), PARENT_DEAD1.G3 (GND1__2), PARENT_DEAD1.G4 (GND1__3), PARENT_DEAD1.G5 (GND2), PARENT_DEAD1.G6 (GND2__1), PARENT_DEAD1.G7 (GND2__2), PARENT_DEAD1.G8 (GND2__3), C100.2, C101.2, C102.2, C103.2, C104.1, C105.2, C106.2, C107.2, C108.2, C109.2, C110.2, C111.2, C112.2, C113.2, C114.2, C115.2, C116.2, C117.2, C118.2, C119.2, C120.2, C121.2, C96.2, C97.2, C98.2, C99.2, LQFP100_DATA_1.23, LQFP100_DATA_1.G1 (GND), LQFP100_DATA_1.G2 (GND__1), LQFP100_DATA_1.G3 (GND__2), LQFP100_DATA_1.G4 (GND__3), LQFP100_DATA_1.G5 (GND__4), LQFP100_DATA_1.G6 (GND__5), LQFP100_DATA_1.G7 (GND__6), LQFP100_DATA_1.G8 (GND__7), LQFP100_DEAD_1.G1 (GND), LQFP100_DEAD_1.G2 (GND__1), LQFP100_DEAD_1.G3 (GND__2), LQFP100_DEAD_1.G4 (GND__3), LQFP100_DEAD_1.G5 (GND__4), LQFP100_DEAD_1.G6 (GND__5), LQFP100_DEAD_1.G7 (GND__6), LQFP100_DEAD_1.G8 (GND__7), LQFP64_DATA_1.19, LQFP64_DATA_1.G1 (GND), LQFP64_DATA_1.G2 (GND__1), LQFP64_DATA_1.G3 (GND__2), LQFP64_DATA_1.G4 (GND__3), LQFP64_DATA_1.G5 (GND__4), LQFP64_DATA_1.G6 (GND__5), LQFP64_DATA_1.G7 (GND__6), LQFP64_DATA_1.G8 (GND__7), LQFP64_DEAD_1.G1 (GND), LQFP64_DEAD_1.G2 (GND__1), LQFP64_DEAD_1.G3 (GND__2), LQFP64_DEAD_1.G4 (GND__3), LQFP64_DEAD_1.G5 (GND__4), LQFP64_DEAD_1.G6 (GND__5), LQFP64_DEAD_1.G7 (GND__6), LQFP64_DEAD_1.G8 (GND__7)
- net TGT_PWR: now also LQFP100_DATA_1.87, LQFP64_DATA_1.87
- new net 100_1: J5.1 (Pin_1), J_SOCKET_100_1.1
- new net 100_12: J6.6 (Pin_6), J_SOCKET_100_1.12
- new net 100_13: J5.7 (Pin_7), J_SOCKET_100_1.13
- new net 100_15: J5.8 (Pin_8), J_SOCKET_100_1.15
- new net 100_16: J6.8 (Pin_8), J_SOCKET_100_1.16
- new net 100_17: J5.9 (Pin_9), J_SOCKET_100_1.17
- new net 100_18: J6.9 (Pin_9), J_SOCKET_100_1.18
- new net 100_2: J6.1 (Pin_1), J_SOCKET_100_1.2
- new net 100_23: J5.12 (Pin_12), J_SOCKET_100_1.23
- new net 100_24: J6.12 (Pin_12), J_SOCKET_100_1.24
- new net 100_25: J5.13 (Pin_13), J_SOCKET_100_1.25
- new net 100_26: J6.13 (Pin_13), J_SOCKET_100_1.26
- new net 100_29: J5.15 (Pin_15), J_SOCKET_100_1.29
- new net 100_3: J5.2 (Pin_2), J_SOCKET_100_1.3
- new net 100_30: J6.15 (Pin_15), J_SOCKET_100_1.30
- new net 100_31: J5.16 (Pin_16), J_SOCKET_100_1.31
- new net 100_32: J6.16 (Pin_16), J_SOCKET_100_1.32
- new net 100_33: J5.17 (Pin_17), J_SOCKET_100_1.33
- new net 100_34: J6.17 (Pin_17), J_SOCKET_100_1.34
- new net 100_35: J5.18 (Pin_18), J_SOCKET_100_1.35
- new net 100_36: J6.18 (Pin_18), J_SOCKET_100_1.36
- new net 100_37: J5.19 (Pin_19), J_SOCKET_100_1.37
- new net 100_38: J6.19 (Pin_19), J_SOCKET_100_1.38
- new net 100_39: J5.20 (Pin_20), J_SOCKET_100_1.39
- new net 100_4: J6.2 (Pin_2), J_SOCKET_100_1.4
- new net 100_40: J6.20 (Pin_20), J_SOCKET_100_1.40
- new net 100_41: J5.21 (Pin_21), J_SOCKET_100_1.41
- new net 100_42: J6.21 (Pin_21), J_SOCKET_100_1.42
- new net 100_43: C114.1, J5.22 (Pin_22), J_SOCKET_100_1.43
- new net 100_44: J6.22 (Pin_22), J_SOCKET_100_1.44
- new net 100_45: J5.23 (Pin_23), J_SOCKET_100_1.45
- new net 100_46: J6.23 (Pin_23), J_SOCKET_100_1.46
- new net 100_47: J5.24 (Pin_24), J_SOCKET_100_1.47
- new net 100_48: C109.1, J6.24 (Pin_24), J_SOCKET_100_1.48
- new net 100_5: J5.3 (Pin_3), J_SOCKET_100_1.5
- new net 100_51: J7.1 (Pin_1), J_SOCKET_100_1.51
- new net 100_52: J8.1 (Pin_1), J_SOCKET_100_1.52
- new net 100_53: J7.2 (Pin_2), J_SOCKET_100_1.53
- new net 100_54: J8.2 (Pin_2), J_SOCKET_100_1.54
- new net 100_55: J7.3 (Pin_3), J_SOCKET_100_1.55
- new net 100_56: C117.1, J8.3 (Pin_3), J_SOCKET_100_1.56
- new net 100_57: J7.4 (Pin_4), J_SOCKET_100_1.57
- new net 100_58: J8.4 (Pin_4), J_SOCKET_100_1.58
- new net 100_59: J7.5 (Pin_5), J_SOCKET_100_1.59
- new net 100_60: J8.5 (Pin_5), J_SOCKET_100_1.60
- new net 100_61: J7.6 (Pin_6), J_SOCKET_100_1.61
- new net 100_62: C118.1, J8.6 (Pin_6), J_SOCKET_100_1.62
- new net 100_63: J7.7 (Pin_7), J_SOCKET_100_1.63
- new net 100_64: J8.7 (Pin_7), J_SOCKET_100_1.64
- new net 100_65: J7.8 (Pin_8), J_SOCKET_100_1.65
- new net 100_66: J8.8 (Pin_8), J_SOCKET_100_1.66
- new net 100_67: J7.9 (Pin_9), J_SOCKET_100_1.67
- new net 100_7: J5.4 (Pin_4), J_SOCKET_100_1.7
- new net 100_70: J8.10 (Pin_10), J_SOCKET_100_1.70
- new net 100_71: J7.11 (Pin_11), J_SOCKET_100_1.71
- new net 100_73: C119.1, J7.12 (Pin_12), J_SOCKET_100_1.73
- new net 100_77: J7.14 (Pin_14), J_SOCKET_100_1.77
- new net 100_78: J8.14 (Pin_14), J_SOCKET_100_1.78
- new net 100_79: J7.15 (Pin_15), J_SOCKET_100_1.79
- new net 100_8: J6.4 (Pin_4), J_SOCKET_100_1.8
- new net 100_80: J8.15 (Pin_15), J_SOCKET_100_1.80
- new net 100_81: J7.16 (Pin_16), J_SOCKET_100_1.81
- new net 100_82: J8.16 (Pin_16), J_SOCKET_100_1.82
- new net 100_83: J7.17 (Pin_17), J_SOCKET_100_1.83
- new net 100_84: J8.17 (Pin_17), J_SOCKET_100_1.84
- new net 100_85: J7.18 (Pin_18), J_SOCKET_100_1.85
- new net 100_86: J8.18 (Pin_18), J_SOCKET_100_1.86
- new net 100_87: J7.19 (Pin_19), J_SOCKET_100_1.87
- new net 100_88: J8.19 (Pin_19), J_SOCKET_100_1.88
- new net 100_89: J7.20 (Pin_20), J_SOCKET_100_1.89
- new net 100_9: J5.5 (Pin_5), J_SOCKET_100_1.9
- new net 100_90: J8.20 (Pin_20), J_SOCKET_100_1.90
- new net 100_91: J7.21 (Pin_21), J_SOCKET_100_1.91
- new net 100_92: J8.21 (Pin_21), J_SOCKET_100_1.92
- new net 100_93: J7.22 (Pin_22), J_SOCKET_100_1.93
- new net 100_95: J7.23 (Pin_23), J_SOCKET_100_1.95
- new net 100_96: J8.23 (Pin_23), J_SOCKET_100_1.96
- new net 100_97: J7.24 (Pin_24), J_SOCKET_100_1.97
- new net 100_98: J8.24 (Pin_24), J_SOCKET_100_1.98
- new net 64_10: J2.5 (Pin_5), J_SOCKET_64_1.10
- new net 64_11: J1.6 (Pin_6), J_SOCKET_64_1.11
- new net 64_14: J2.7 (Pin_7), J_SOCKET_64_1.14
- new net 64_15: J1.8 (Pin_8), J_SOCKET_64_1.15
- new net 64_16: J2.8 (Pin_8), J_SOCKET_64_1.16
- new net 64_2: J2.1 (Pin_1), J_SOCKET_64_1.2
- new net 64_20: J2.10 (Pin_10), J_SOCKET_64_1.20
- new net 64_21: J1.11 (Pin_11), J_SOCKET_64_1.21
- new net 64_22: J2.11 (Pin_11), J_SOCKET_64_1.22
- new net 64_23: J1.12 (Pin_12), J_SOCKET_64_1.23
- new net 64_24: J2.12 (Pin_12), J_SOCKET_64_1.24
- new net 64_25: J1.13 (Pin_13), J_SOCKET_64_1.25
- new net 64_26: J2.13 (Pin_13), J_SOCKET_64_1.26
- new net 64_27: J1.14 (Pin_14), J_SOCKET_64_1.27
- new net 64_28: J2.14 (Pin_14), J_SOCKET_64_1.28
- new net 64_29: J1.15 (Pin_15), J_SOCKET_64_1.29
- new net 64_3: J1.2 (Pin_2), J_SOCKET_64_1.3
- new net 64_30: C102.1, J2.15 (Pin_15), J_SOCKET_64_1.30
- new net 64_34: J4.1 (Pin_1), J_SOCKET_64_1.34
- new net 64_35: J3.2 (Pin_2), J_SOCKET_64_1.35
- new net 64_36: J4.2 (Pin_2), J_SOCKET_64_1.36
- new net 64_37: J3.3 (Pin_3), J_SOCKET_64_1.37
- new net 64_38: J4.3 (Pin_3), J_SOCKET_64_1.38
- new net 64_39: J3.4 (Pin_4), J_SOCKET_64_1.39
- new net 64_4: J2.2 (Pin_2), J_SOCKET_64_1.4
- new net 64_40: J4.4 (Pin_4), J_SOCKET_64_1.40
- new net 64_41: J3.5 (Pin_5), J_SOCKET_64_1.41
- new net 64_44: J4.6 (Pin_6), J_SOCKET_64_1.44
- new net 64_45: J3.7 (Pin_7), J_SOCKET_64_1.45
- new net 64_5: J1.3 (Pin_3), J_SOCKET_64_1.5
- new net 64_50: J4.9 (Pin_9), J_SOCKET_64_1.50
- new net 64_51: J3.10 (Pin_10), J_SOCKET_64_1.51
- new net 64_52: J4.10 (Pin_10), J_SOCKET_64_1.52
- new net 64_53: J3.11 (Pin_11), J_SOCKET_64_1.53
- new net 64_54: J4.11 (Pin_11), J_SOCKET_64_1.54
- new net 64_55: J3.12 (Pin_12), J_SOCKET_64_1.55
- new net 64_56: J4.12 (Pin_12), J_SOCKET_64_1.56
- new net 64_57: J3.13 (Pin_13), J_SOCKET_64_1.57
- new net 64_58: J4.13 (Pin_13), J_SOCKET_64_1.58
- new net 64_59: J3.14 (Pin_14), J_SOCKET_64_1.59
- new net 64_6: J2.3 (Pin_3), J_SOCKET_64_1.6
- new net 64_61: J3.15 (Pin_15), J_SOCKET_64_1.61
- new net 64_62: J4.15 (Pin_15), J_SOCKET_64_1.62
- new net 64_8: J2.4 (Pin_4), J_SOCKET_64_1.8
- new net 64_9: J1.5 (Pin_5), J_SOCKET_64_1.9
- no-connect marks 676 -> 652
Other:
- note added: "VCAP100 -> 43,48,49,56,62,73 VCAP64 -> 30,31,47"
- note removed: "LQFP100 -> dead socket"
- note removed: "LQFP64 -> dead socket"
- moved on the sheet: C79, C88, C90, C92, C93, C95, DEC1, INV6, J_CARDX_L_1A, J_CARDX_L_1B, LQFP100_SWD1, LQFP100_USART1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

Commit message: lqfp64 targer
Parts:
- removed C106: .1u, Capacitor_SMD:C_0402_1005Metric, symbol Device:C_Small_US
Connections:
- net 100_72: no longer J4.7 (Pin_7), J_SOCKET_64_1.46
- net 100_76: no longer J3.9 (Pin_9), J_SOCKET_64_1.49
- net GND: no longer PARENT_DEAD1.G1 (GND1), PARENT_DEAD1.G2 (GND1__1), PARENT_DEAD1.G3 (GND1__2), PARENT_DEAD1.G4 (GND1__3), PARENT_DEAD1.G5 (GND2), PARENT_DEAD1.G6 (GND2__1), PARENT_DEAD1.G7 (GND2__2), PARENT_DEAD1.G8 (GND2__3)
- net SWDCLK_64 renamed 64_49
- net 64_49: now also J3.9 (Pin_9), J_SOCKET_64_1.49
- net SWDIO_64 renamed 64_46
- net 64_46: now also J4.7 (Pin_7), J_SOCKET_64_1.46
- no-connect marks 652 -> 660
