File: Profile_Switching.kicad_sch (KiCad schematic)
At the start: 140 parts, among them J1 Conn_01x16_Pin, J10 Conn_01x08_Pin, J11 Conn_01x09_Pin, J12 Conn_01x08_Pin, J13 Conn_01x08_Pin, J14 Conn_01x09_Pin, J15 Conn_01x08_Pin, J16 Conn_01x08_Pin, J2 Conn_01x16_Pin, J3 Conn_01x16_Pin, J4 Conn_01x16_Pin, J5 Conn_01x08_Pin, J6 Conn_01x09_Pin, J7 Conn_01x08_Pin, J8 Conn_01x09_Pin, J9 Conn_01x08_Pin

Commit message: Update
Connections:
- net 100_68: no longer LQFP100_USART1.1 (Pin_1)
- net 100_69: no longer LQFP100_USART1.2 (Pin_2)
- net 100_72: no longer LQFP100_SWD1.1 (Pin_1)
- net 100_76: no longer LQFP100_SWD1.2 (Pin_2)
- net 64_42: no longer LQFP64_USART1.1 (Pin_1)
- net 64_43: no longer LQFP64_USART1.2 (Pin_2)
- net LQFP100_PIN_68: now also LQFP100_USART1.1 (Pin_1)
- net LQFP100_PIN_69: now also LQFP100_USART1.2 (Pin_2)
- net LQFP64_PIN_42: now also LQFP64_USART1.1 (Pin_1)
- net LQFP64_PIN_43: now also LQFP64_USART1.2 (Pin_2)
- new net LQFP100_PIN_72: LQFP100_SWD1.1 (Pin_1)
- new net LQFP100_PIN_76: LQFP100_SWD1.2 (Pin_2)
Changed lines of the file:
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@@
 		)
 	)
-	(label "100_76"
+	(label "LQFP100_PIN_76"
 		(at 1012.19 172.72 180)
 		(effects
@@
 		)
 	)
-	(label "100_69"
+	(label "LQFP100_PIN_69"
 		(at 1008.38 140.97 180)
 		(effects
@@
 		)
 	)
-	(label "100_72"
+	(label "LQFP100_PIN_72"
 		(at 1012.19 166.37 180)
 		(effects
@@
 		)
 	)
-	(label "64_43"
+	(label "LQFP64_PIN_43"
 		(at 1066.8 140.97 180)
 		(effects
@@
 		)
 	)
-	(label "64_42"
+	(label "LQFP64_PIN_42"
 		(at 1066.8 134.62 180)
 		(effects
@@
 		)
 	)
-	(label "100_68"
+	(label "LQFP100_PIN_68"
 		(at 1008.38 134.62 180)
 		(effects

Commit message: Update
Parts:
- AND3, AND4, BUF1, BUF10, BUF11, BUF12, BUF2, BUF3, BUF4, BUF5, BUF6, BUF7, BUF8, BUF9, INV4, INV5, INV6, INV7, LD1, LD2, LD3, LD4, LD5, LD6, LD7, LS1, LS2, NAND1, OR1, OR2, OR3, OR4, SPST1, SPST2, SPST3, SPST4: KiLib_Generator (none) -> package/gullwing
- C100, C101, C102, C103, C104, C105, C107, C108, C109, C110, C111, C113, C114, C115, C116, C117, C118, C119, C120, C121, C73, C74, C75, C76, C77, C78, C79, C80, C81, C82, C83, C84, C85, C86, C87, C88, C89, C90, C91, C92, C93, C94, C95, C96, C97, C98, C99, R64, R65, R66, R67, R68, R69, R70, R71, R72, R73, R74, R75, R76, R77, R78, R79, R80, R81, R82, R83, R84, R85, R86, R87, R88, R89, R90: KiLib_Generator (none) -> SMD_2terminal_chip_molded
- J1, J10, J11, J12, J13, J14, J15, J16, J2, J3, J4, J5, J6, J7, J8, J9, LQFP100_SWD1, LQFP100_USART1, LQFP64_SWD1, LQFP64_USART1: KiLib_Generator (none) -> connector/pin_header_socket
Connections:
- net 100_100: now also J14.9 (Pin_9)
- net 100_68: now also LQFP100_USART1.1 (Pin_1)
- net 100_69: now also LQFP100_USART1.2 (Pin_2)
- net 100_72: now also LQFP100_SWD1.1 (Pin_1)
- net 100_76: now also J14.1 (Pin_1), LQFP100_SWD1.2 (Pin_2)
- net 100_79: now also J14.2 (Pin_2)
- net 100_82: now also J14.3 (Pin_3)
- net 100_85: now also J14.4 (Pin_4)
- net 100_88: now also J14.5 (Pin_5)
- net 100_91: now also J14.6 (Pin_6)
- net 100_94: now also J14.7 (Pin_7); no longer J14.3 (Pin_3)
- net 100_97: now also J14.8 (Pin_8)
- net 3V3: no longer LQFP100_DATA_1.65, LQFP64_DATA_1.65
- net 64_42: now also LQFP64_USART1.1 (Pin_1)
- net 64_43: now also LQFP64_USART1.2 (Pin_2)
- net LQFP100_PIN_68: no longer LQFP100_USART1.1 (Pin_1)
- net LQFP100_PIN_69: no longer LQFP100_USART1.2 (Pin_2)
- net LQFP100_PIN_72: no longer LQFP100_SWD1.1 (Pin_1)
- net LQFP100_PIN_76: no longer LQFP100_SWD1.2 (Pin_2)
- net LQFP64_PIN_42: no longer LQFP64_USART1.1 (Pin_1)
- net LQFP64_PIN_43: no longer LQFP64_USART1.2 (Pin_2)
- net TGT_PWR renamed TGT_PWR64
- net TGT_PWR64: no longer LQFP100_DATA_1.87, LQFP100_SWD1.3 (Pin_3)
- new net 3V3_100: LQFP100_DATA_1.65
- new net 3V3_64: LQFP64_DATA_1.65
- new net TGT_PWR100: LQFP100_DATA_1.87, LQFP100_SWD1.3 (Pin_3)

Commit message: cg edits
Parts:
- removed J1, J2, J3, J4: Conn_01x16_Pin, Connector_PinHeader_2.54mm:PinHeader_1x16_P2.54mm_Vertical, symbol Connector:Conn_01x16_Pin
- added J1, J2, J3, J4, J5, J6, J7, J8: Conn_01x08_Pin, Connector_PinHeader_2.54mm:PinHeader_1x08_P2.54mm_Vertical, symbol Connector:Conn_01x08_Pin
- renumbered C107 to C106, C108 to C107, C109 to C108, C110 to C109, C111 to C110, C112 to C111, C113 to C112, C114 to C113, C115 to C114, C116 to C115, C117 to C116, C118 to C117, C119 to C118, C120 to C119, C121 to C120, J6 to J10, J9 to J11, J5 to J12, J10 to J13, J7 to J14, J14 to J15, J11 to J16, J15 to J17, J12 to J18, J16 to J19, J13 to J20, J8 to J9
Connections:
- net 64_1: now also J3.4 (Pin_4)
- net 64_10: now also J3.5 (Pin_5)
- net 64_11: now also J4.8 (Pin_8)
- net 64_12: now also J3.7 (Pin_7)
- net 64_13: now also J4.5 (Pin_5)
- net 64_14: now also J4.7 (Pin_7)
- net 64_15: now also J3.6 (Pin_6)
- net 64_16: now also J4.6 (Pin_6)
- net 64_17: now also J1.5 (Pin_5)
- net 64_18: now also J1.6 (Pin_6)
- net 64_19: now also J1.7 (Pin_7)
- net 64_2: now also J3.3 (Pin_3)
- net 64_20: now also J2.6 (Pin_6)
- net 64_21: now also J2.8 (Pin_8)
- net 64_22: now also J1.8 (Pin_8)
- net 64_23: now also J2.5 (Pin_5)
- net 64_24: now also J2.7 (Pin_7)
- net 64_25: now also J1.1 (Pin_1)
- net 64_26: now also J2.4 (Pin_4)
- net 64_27: now also J1.4 (Pin_4)
- net 64_28: now also J1.2 (Pin_2)
- net 64_29: now also J2.3 (Pin_3)
- net 64_3: now also J3.2 (Pin_2)
- net 64_30: now also J2.2 (Pin_2)
- net 64_31: now also J2.1 (Pin_1)
- net 64_32: now also J1.3 (Pin_3)
- net 64_34: now also J7.7 (Pin_7)
- net 64_35: now also J7.6 (Pin_6), J7.8 (Pin_8)
- net 64_36: now also J8.5 (Pin_5)
- net 64_37: now also J8.3 (Pin_3)
- net 64_38: now also J8.7 (Pin_7)
- net 64_39: now also J8.4 (Pin_4)
- net 64_4: now also J4.3 (Pin_3)
- net 64_40: now also J8.2 (Pin_2)
- net 64_41: now also J8.6 (Pin_6)
- net 64_42: now also J7.5 (Pin_5)
- net 64_43: now also J8.8 (Pin_8)
- net 64_44: now also J8.1 (Pin_1)
- net 64_45: now also J7.4 (Pin_4)
- net 64_46: now also J7.2 (Pin_2)
- net 64_47: now also J7.1 (Pin_1)
- net 64_48: now also J7.3 (Pin_3)
- net 64_49: now also J6.1 (Pin_1)
- net 64_5: now also J4.2 (Pin_2)
- net 64_50: now also J5.4 (Pin_4)
- net 64_51: now also J5.2 (Pin_2)
- net 64_52: now also J6.2 (Pin_2)
- net 64_53: now also J5.3 (Pin_3)
- net 64_54: now also J5.1 (Pin_1)
- net 64_55: now also J6.3 (Pin_3)
- net 64_56: now also J6.8 (Pin_8)
- net 64_57: now also J5.8 (Pin_8)
- net 64_58: now also J6.4 (Pin_4)
- net 64_59: now also J6.7 (Pin_7)
- net 64_6: now also J3.1 (Pin_1)
- net 64_60: now also J5.7 (Pin_7)
- net 64_61: now also J6.5 (Pin_5)
- net 64_62: now also J6.6 (Pin_6)
- net 64_63: now also J5.6 (Pin_6)
- net 64_64: now also J5.5 (Pin_5)
- net 64_7: now also J4.4 (Pin_4)
- net 64_8: now also J4.1 (Pin_1)
- net 64_9: now also J3.8 (Pin_8)
- net GND: no longer LQFP100_DEAD_1.G1 (GND), LQFP100_DEAD_1.G2 (GND__1), LQFP100_DEAD_1.G3 (GND__2), LQFP100_DEAD_1.G4 (GND__3), LQFP100_DEAD_1.G5 (GND__4), LQFP100_DEAD_1.G6 (GND__5), LQFP100_DEAD_1.G7 (GND__6), LQFP100_DEAD_1.G8 (GND__7), LQFP64_DEAD_1.G1 (GND), LQFP64_DEAD_1.G2 (GND__1), LQFP64_DEAD_1.G3 (GND__2), LQFP64_DEAD_1.G4 (GND__3), LQFP64_DEAD_1.G5 (GND__4), LQFP64_DEAD_1.G6 (GND__5), LQFP64_DEAD_1.G7 (GND__6), LQFP64_DEAD_1.G8 (GND__7)
- net TGT_PWR100: now also LQFP100_USART1.3 (Pin_3)
- net TGT_PWR64: no longer LQFP100_USART1.3 (Pin_3)
- net 3V3_64: no longer names the net of LQFP64_DATA_1.65
- no-connect marks 660 -> 677
Other:
- note removed: "USART/BOOT0 - LQFP100"

Commit message: bom
Parts:
- removed C106, C108, C113, C116, C117, C118: 2.2u, Capacitor_SMD:C_0603_1608Metric, symbol Device:C_Small_US
- removed C107, C109, C110, C111, C112, C114, C115, C119, C120: .1u, Capacitor_SMD:C_0402_1005Metric, symbol Device:C_Small_US
- removed J10, J15, J16, J9: Conn_01x09_Pin, Connector_PinHeader_2.54mm:PinHeader_1x09_P2.54mm_Vertical, symbol Connector:Conn_01x09_Pin
- removed J11, J12, J13, J14, J17, J18, J19, J20: Conn_01x08_Pin, Connector_PinHeader_2.54mm:PinHeader_1x08_P2.54mm_Vertical, symbol Connector:Conn_01x08_Pin
- removed J_SOCKET_100_1: IC51-1004-809, MyFootprints:YAMAICHI_IC51-1004-809, symbol MySymbols:IC51-1004-809
- removed LQFP100_DATA_1, LQFP100_DEAD_1, LQFP64_DEAD_1: QTH-060-01-X-D-A, MyFootprints:SAMTEC_QTH-060-01-X-D-A, symbol MySymbols:QTH-060-01-X-D-A
- removed LQFP100_SWD1, LQFP100_USART1: Conn_01x04_Pin, Connector_PinHeader_2.54mm:PinHeader_1x04_P2.54mm_Vertical, symbol Connector:Conn_01x04_Pin
- removed PARENT_DEAD1: QSH-060-01-X-D-A, footprints2:SAMTEC_QSH-060-01-X-D-A, symbol MySymbols:QTH-060-03-X-D-A
Connections:
- no-connect marks 677 -> 195
Other:
- note removed: "Dead Sockets"
- note removed: "Parent Board -> dead socket"
- note removed: "VCAP100 -> 43,48,49,56,62,73 VCAP64 -> 30,31,47"
