File: pcbfiles.kicad_pcb (KiCad board)
At the start: 4 copper layers, 271.1 x 184.3 mm, 406 parts, among them J1 Conn_01x08_Pin, J10 Conn_01x08_Pin, J11 Conn_01x09_Pin, J12 Conn_01x08_Pin, J13 Conn_01x08_Pin, J14 Conn_01x09_Pin, J15 Conn_01x08_Pin, J16 Conn_01x08_Pin, J2 Conn_01x08_Pin, J3 Conn_01x08_Pin, J4 Conn_01x08_Pin, J5 Conn_01x08_Pin, J6 Conn_01x08_Pin, J6 Conn_01x09_Pin, J7 Conn_01x08_Pin, J8 Conn_01x08_Pin, J8 Conn_01x09_Pin, J9 Conn_01x08_Pin, Y1 Crystal_GND24

Commit message: final cuts
dfds
Parts:
- removed 39, 77, 78, 79, 80: , 
- added ?: , , F.Cu at (445.6, 106.5)
- added ?: , , F.Cu at (322.0, 181.9)
- added ?: , , F.Cu at (445.6, 195.5)
- added ?: , , F.Cu at (445.6, 181.9)
- added ?: , , F.Cu at (445.6, 281.0)
- added ?: , , F.Cu at (322.0, 106.6)
- added ?: , , F.Cu at (322.0, 281.0)
- added ?: , , F.Cu at (322.0, 195.5)
- moved LQFP64_DEAD_1 101.6 mm to (436.3, 137.0)
- moved LQFP100_DEAD_1 84.3 mm to (439.2, 236.0), turned to -90 degrees
- moved PARENT_DEAD1 69.1 mm to (296.7, 148.7), turned to -90 degrees
- moved C100 20.4 mm to (366.5, 151.6)
- moved C101 20.4 mm to (377.0, 142.8)
- moved C102 20.4 mm to (373.1, 133.5)
- moved C105 20.4 mm to (351.1, 142.8)
- moved C98 20.4 mm to (370.1, 142.8)
- moved J4 20.4 mm to (354.6, 168.2)
- moved J5 20.4 mm to (333.6, 131.3)
- moved J6 20.4 mm to (327.9, 131.3)
- moved J7 20.4 mm to (355.4, 114.6)
- moved J_SOCKET_64_1 20.4 mm to (364.0, 138.6)
- moved C103 20.4 mm to (368.3, 125.7)
- moved C104 20.4 mm to (358.8, 127.5)
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Other:
- board size 271.1 x 184.3 mm -> 271.1 x 182.6 mm
