File: pcbfiles.kicad_pcb (KiCad board)
At the start: 4 copper layers, 271.1 x 182.6 mm, 406 parts, among them J1 Conn_01x08_Pin, J10 Conn_01x08_Pin, J11 Conn_01x09_Pin, J12 Conn_01x08_Pin, J13 Conn_01x08_Pin, J14 Conn_01x09_Pin, J15 Conn_01x08_Pin, J16 Conn_01x08_Pin, J2 Conn_01x08_Pin, J3 Conn_01x08_Pin, J4 Conn_01x08_Pin, J5 Conn_01x08_Pin, J6 Conn_01x08_Pin, J6 Conn_01x09_Pin, J7 Conn_01x08_Pin, J8 Conn_01x08_Pin, J8 Conn_01x09_Pin, J9 Conn_01x08_Pin, Y1 Crystal_GND24

Commit message: meow v2
Parts:
- turned LQFP100_DATA_1 to -90 degrees
Routing:
- net /Profile_Switching/100_75: track 98.3 -> 36.1 mm, vias 1 -> 0
- net unconnected-(LQFP100_DATA_1-Pad64): track 0.00 -> 31.1 mm
- net /Profile_Switching/100_74: track 64.5 -> 38.9 mm, vias 1 -> 0
- net /Profile_Switching/100_11: track 163.5 -> 141.2 mm
- net /Profile_Switching/100_14: track 181.0 -> 159.2 mm
- net /Profile_Switching/100_99: track 138.3 -> 116.9 mm
- net /Profile_Switching/100_94: track 107.6 -> 87.3 mm
- net /Profile_Switching/100_22: track 144.7 -> 127.9 mm
- net /Profile_Switching/100_27: track 138.5 -> 122.9 mm, vias 1 -> 0
- net /Profile_Switching/100_69: track 79.8 -> 64.8 mm, vias 3 -> 2
- net /Profile_Switching/100_6: track 193.4 -> 178.5 mm
- net /Profile_Switching/100_100: track 151.4 -> 137.5 mm
- net /Profile_Switching/100_20: track 209.1 -> 197.7 mm, vias 1 -> 0
- net /Profile_Switching/100_49: track 91.0 -> 80.9 mm, vias 3 -> 2
- net /Profile_Switching/100_68: track 93.8 -> 85.0 mm, vias 2 -> 1
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