File: pcbfiles.kicad_pcb (KiCad board)
At the start: 4 copper layers, 218.4 x 192.8 mm, 391 parts, among them J1 Conn_01x08_Pin, J10 Conn_01x08_Pin, J11 Conn_01x09_Pin, J12 Conn_01x08_Pin, J13 Conn_01x08_Pin, J14 Conn_01x09_Pin, J15 Conn_01x08_Pin, J16 Conn_01x08_Pin, J2 Conn_01x08_Pin, J3 Conn_01x08_Pin, J4 Conn_01x08_Pin, J5 Conn_01x08_Pin, J6 Conn_01x08_Pin, J6 Conn_01x09_Pin, J7 Conn_01x08_Pin, J8 Conn_01x08_Pin, J8 Conn_01x09_Pin, J9 Conn_01x08_Pin, Y1 Crystal_GND24

Commit message: final impelementation
Parts:
- removed the 43 at (293.6, 125.6)
- removed the 44 at (293.6, 129.6)
- removed the 45 at (293.6, 133.6)
- removed the 46 at (293.6, 137.6)
- removed the 47 at (293.6, 141.6)
- removed the 48 at (293.6, 145.6)
- removed the 49 at (293.6, 149.6)
- removed the 50 at (293.6, 153.6)
- removed the 51 at (293.6, 157.6)
- removed the 52 at (293.6, 161.6)
- removed the 53 at (293.6, 165.6)
- removed the 54 at (293.6, 169.6)
- removed the 55 at (293.6, 173.6)
- removed the 56 at (293.6, 177.6)
- removed the 57 at (293.6, 181.6)
- removed the 58 at (293.6, 185.6)
- removed the 59 at (293.4, 189.5)
- removed the 60 at (293.6, 193.6)
- removed the 61 at (293.6, 197.6)
- removed the 62 at (293.6, 201.6)
- removed 63 (x2), 64 (x2), 65 (x2), 66, 67, 68, 69, 70, 71, 72, 73, 74, 75: , 
- removed C107, C109, C114, C117, C118, C119: 2.2u, Capacitor_SMD:C_0603_1608Metric
- removed C108, C110, C111, C112, C113, C115, C116, C120, C121: .1u, Capacitor_SMD:C_0402_1005Metric
- removed J10, J12, J13, J15, J16, J9: Conn_01x08_Pin, Connector_PinHeader_2.54mm:PinHeader_1x08_P2.54mm_Vertical
- removed J11, J14: Conn_01x09_Pin, Connector_PinHeader_2.54mm:PinHeader_1x09_P2.54mm_Vertical
- removed the J5 at (381.9, 246.8)
- removed the J6 at (378.1, 248.1)
- removed the J7 at (385.7, 246.8)
- removed the J8 at (361.6, 211.3)
- removed J_SOCKET_100_1: IC51-1004-809, MyFootprints:YAMAICHI_IC51-1004-809
- removed LQFP100_DATA_1: QTH-060-01-X-D-A, MyFootprints:SAMTEC_QTH-060-01-X-D-A
- removed the REF** at (392.4, 184.6)
- removed the REF** at (392.4, 283.0)
- removed the REF** at (392.4, 99.4)
- removed the REF** at (392.4, 197.9)
- removed the SWD at (318.9, 261.6)
- removed the USART1 at (325.3, 261.5)
- added 62: , , F.Cu at (271.0, 259.7)
- added 62: , , F.Cu at (274.7, 259.9)
- added REF**: MountingHole_3.2mm_M3, MountingHole:MountingHole_3.2mm_M3, F.Cu at (260.3, 328.4)
- added REF**: MountingHole_3.2mm_M3, MountingHole:MountingHole_3.2mm_M3, F.Cu at (260.1, 272.4)
- moved C100 197.2 mm to (228.0, 286.5)
- moved C104 197.2 mm to (235.7, 310.5)
- moved C99 197.2 mm to (234.7, 286.6)
- moved J3 197.2 mm to (239.9, 275.9)
- moved J6 197.2 mm to (266.6, 306.8)
- moved USART1 197.2 mm to (209.6, 318.4)
- moved C101 197.2 mm to (217.4, 295.3)
- moved C103 197.2 mm to (226.2, 312.4)
- moved C105 197.2 mm to (243.4, 295.3)
- moved C96 197.2 mm to (217.5, 302.9)
- moved C97 197.2 mm to (224.7, 304.4)
- moved C98 197.2 mm to (224.4, 295.2)
- moved J1 197.2 mm to (207.0, 307.7)
- moved J2 197.2 mm to (200.8, 307.8)
- moved J4 197.2 mm to (239.8, 269.9)
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- renumbered LQFP64_USART1 to USART1
Routing:
- net /Profile_Switching/100_20: track 190.8 -> 0.00 mm, vias 1 -> 0
- net /Profile_Switching/100_6: track 171.9 -> 0.00 mm, vias 4 -> 0
- net /Profile_Switching/100_11: track 169.2 -> 0.00 mm, vias 4 -> 0
- net /Profile_Switching/100_22: track 168.9 -> 0.00 mm, vias 3 -> 0
- net /Profile_Switching/100_21: track 167.9 -> 0.00 mm, vias 1 -> 0
- net /Profile_Switching/100_10: track 166.8 -> 0.00 mm, vias 3 -> 0
- net /Profile_Switching/100_14: track 164.6 -> 0.00 mm, vias 4 -> 0
- net /Profile_Switching/100_99: track 156.6 -> 0.00 mm, vias 5 -> 0
- net /Profile_Switching/100_19: track 143.7 -> 0.00 mm, vias 3 -> 0
- net /Profile_Switching/100_100: track 124.0 -> 0.00 mm, vias 3 -> 0
- net /Profile_Switching/100_28: track 121.6 -> 0.00 mm, vias 2 -> 0
- net /Profile_Switching/100_94: track 104.4 -> 0.00 mm, vias 3 -> 0
- net /Profile_Switching/100_27: track 98.1 -> 0.00 mm, vias 3 -> 0
- net /Profile_Switching/100_68: track 93.9 -> 0.00 mm, vias 1 -> 0
- net /Profile_Switching/100_50: track 93.0 -> 0.00 mm, vias 4 -> 0
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- removed copper zone on In2.Cu, net /Profile_Switching/TGT_PWR100
- removed copper zone on B.Cu, net GND100
- removed copper zone on F.Cu, net GND100
- removed copper zone on In1.Cu, net GND100
Other:
- board size 218.4 x 192.8 mm -> 113.5 x 212.5 mm
- board text added: "CYBERDECK PARENT BOARD"
- board text added: "CyberDeck supports 1V8/3V3 Target STM32F MCU's. Toggle switches to set power supply and use the TARGET_PWR button to enable victim power. Toggle both switches for AUTO toggle through 1V8 and 3V3 power until target MCU is identified. If the board is not identified, Target PWR is set to OFF and the target board is simply a breakout board and should be used UNPLUGGED FROM THE CyberDeck to avoid dama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"
- board text added: "INSTRUCTIONS 1. USB-C Power (5V/1.5A capable) or 18650 3.6V battery required 2. Insert Target MCU into corresponding target board socket connector. 3. Plug in target board to CyberDeck socket. 4. Set desired POWER SUPPLY settings. Push TARGET_PWR_EN. 5. Wait for CyberDeck to identify target MCU on LCD Screen. 6. Use breakout pins on Target Boards to access target."
- board text added: "RevA"
- board text added: "STM32F LQFP64 TARGET CHIP"
- board text added: "VREF"
- board text removed: "100"
- board text removed: "2 5 8 11 14 17 20 23"
- board text removed: "27 30 33 36 39 42 45 48"
- board text removed: "66"
- board text removed: "67"
- board text removed: "69"
- board text removed: "70"
- board text removed: "72"
- board text removed: "73"
- board text removed: "74 71 68 65 62 59 56 53"
- board text removed: "75"
- board text removed: "76"
- board text removed: "78"
- board text removed: "79"
- board text removed: "81"
- board text removed: "82"
- board text removed: "84"
- board text removed: "85"
- board text removed: "87"
- board text removed: "88"
- board text removed: "90"
- board text removed: "91"
- board text removed: "93"
- board text removed: "94"
- board text removed: "96"
- board text removed: "97"
- board text removed: "98 95 92 89 86 83 80 77"
- board text removed: "99"
- board text removed: "PWR"
