File: FINALE SAUCE.kicad_pcb (KiCad board)
At the start: 4 copper layers, 218.4 x 192.8 mm, 391 parts, among them J1 Conn_01x08_Pin, J10 Conn_01x08_Pin, J11 Conn_01x09_Pin, J12 Conn_01x08_Pin, J13 Conn_01x08_Pin, J14 Conn_01x09_Pin, J15 Conn_01x08_Pin, J16 Conn_01x08_Pin, J2 Conn_01x08_Pin, J3 Conn_01x08_Pin, J4 Conn_01x08_Pin, J5 Conn_01x08_Pin, J6 Conn_01x08_Pin, J6 Conn_01x09_Pin, J7 Conn_01x08_Pin, J8 Conn_01x08_Pin, J8 Conn_01x09_Pin, J9 Conn_01x08_Pin, Y1 Crystal_GND24

Commit message: bom
Parts:
- removed C107, C109, C114, C117, C118, C119: 2.2u, Capacitor_SMD:C_0603_1608Metric
- removed C108, C110, C111, C112, C113, C115, C116, C120, C121: .1u, Capacitor_SMD:C_0402_1005Metric
- removed J10, J12, J13, J15, J16, J9: Conn_01x08_Pin, Connector_PinHeader_2.54mm:PinHeader_1x08_P2.54mm_Vertical
- removed J11, J14: Conn_01x09_Pin, Connector_PinHeader_2.54mm:PinHeader_1x09_P2.54mm_Vertical
- removed the J5 at (381.9, 246.8)
- removed the J6 at (378.1, 248.1)
- removed the J7 at (385.7, 246.8)
- removed the J8 at (361.6, 211.3)
- removed J_SOCKET_100_1: IC51-1004-809, MyFootprints:YAMAICHI_IC51-1004-809
- removed LQFP100_DATA_1: QTH-060-01-X-D-A, MyFootprints:SAMTEC_QTH-060-01-X-D-A
- removed the REF** at (392.4, 283.0)
- removed the REF** at (392.4, 197.9)
- removed the SWD at (318.9, 261.6)
- removed USART1: Conn_01x04_Pin, Connector_PinHeader_2.54mm:PinHeader_1x04_P2.54mm_Vertical
Routing:
- net /Profile_Switching/100_20: track 190.8 -> 0.00 mm, vias 1 -> 0
- net /Profile_Switching/100_6: track 171.9 -> 0.00 mm, vias 4 -> 0
- net /Profile_Switching/100_11: track 169.2 -> 0.00 mm, vias 4 -> 0
- net /Profile_Switching/100_22: track 168.9 -> 0.00 mm, vias 3 -> 0
- net /Profile_Switching/100_21: track 167.9 -> 0.00 mm, vias 1 -> 0
- net /Profile_Switching/100_10: track 166.8 -> 0.00 mm, vias 3 -> 0
- net /Profile_Switching/100_14: track 164.6 -> 0.00 mm, vias 4 -> 0
- net /Profile_Switching/100_99: track 156.6 -> 0.00 mm, vias 5 -> 0
- net /Profile_Switching/100_19: track 143.7 -> 0.00 mm, vias 3 -> 0
- net /Profile_Switching/100_100: track 124.0 -> 0.00 mm, vias 3 -> 0
- net /Profile_Switching/100_28: track 121.6 -> 0.00 mm, vias 2 -> 0
- net /Profile_Switching/100_94: track 104.4 -> 0.00 mm, vias 3 -> 0
- net /Profile_Switching/100_27: track 98.1 -> 0.00 mm, vias 3 -> 0
- net /Profile_Switching/100_68: track 93.9 -> 0.00 mm, vias 1 -> 0
- net /Profile_Switching/100_50: track 93.0 -> 0.00 mm, vias 4 -> 0
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- removed copper zone on In2.Cu, net /Profile_Switching/TGT_PWR100
- removed copper zone on B.Cu, net GND100
- removed copper zone on F.Cu, net GND100
- removed copper zone on In1.Cu, net GND100
