File: untitled.kicad_sch (KiCad schematic)
At the start: 130 parts

Commit message: finished routing
//TODO
-> add mechanical support
-> daughter board
-> recheck nodes/conections
-> silk screen
Parts:
- renumbered C12 to C11, C13 to C12, C11 to C13
Connections:
- net 3V3: now also R41.1; no longer R41.2
- net at 3.3V_EN1.3: now also R41.2; no longer R41.1
Other:
- moved on the sheet: BAT1, BAT_CHG1, BAT_SET1, BOOST1, C1, C11, C12, C14, C16, C2, C6, CHGR1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

Commit message: Update
Parts:
- AND1, AND2, BOOST1, INV1, INV2, INV3, OVP1, U-ESD1: KiLib_Generator (none) -> package/gullwing
- BAT_CHG1, BAT_SET1, C1, C10, C11, C12, C13, C14, C15, C16, C17, C18, C19, C2, C20, C21, C22, C23, C24, C25, C26, C27, C28, C29, C3, C30, C31, C32, C33, C34, C35, C36, C37, C38, C39, C4, C40, C41, C42, C43, C44, C45, C46, C47, C48, C49, C5, C6, C7, C8, C9, FLT1, R1, R10, R11, R12, R13, R14, R15, R16, R17, R18, R19, R2, R20, R21, R22, R23, R24, R25, R26, R27, R28, R29, R3, R30, R31, R32, R33, R34, R35, R36, R37, R38, R39, R4, R40, R41, R42, R43, R44, R45, R46, R47, R48, R5, R6, R7, R8, R9, TRGT_PWR1: KiLib_Generator (none) -> SMD_2terminal_chip_molded
- CHGR1: KiLib_Generator (none) -> package/no_lead
- L_BK1, L_BST1: KiLib_Generator (none) -> inductor/SMD

Commit message: cg edits
Parts:
- renumbered TRGT_PWR1 to PWR1
Changed lines of the file:
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@@
 		(dnp no)
 		(fields_autoplaced yes)
-		(property "Reference" "TRGT_PWR1"
+		(property "Reference" "PWR1"
 			(at 420.6875 473.71 0)
 			(show_name no)
@@
 			(project "CG Files"
 				(path "/bab4cc86-0c89-4bf5-848e-e99340a6180d/074ec3ee-4318-401c-b0e4-fc01472c8356"
-					(reference "TRGT_PWR1")
+					(reference "PWR1")
 					(unit 1)
 				)
