File: _restore_backup_2026-07-09T15-35-08-739/Profile_Switching.kicad_sch (KiCad schematic)
At the start: 140 parts, among them J1 Conn_01x16_Pin, J10 Conn_01x08_Pin, J11 Conn_01x09_Pin, J12 Conn_01x08_Pin, J13 Conn_01x08_Pin, J14 Conn_01x09_Pin, J15 Conn_01x08_Pin, J16 Conn_01x08_Pin, J2 Conn_01x16_Pin, J3 Conn_01x16_Pin, J4 Conn_01x16_Pin, J5 Conn_01x08_Pin, J6 Conn_01x09_Pin, J7 Conn_01x08_Pin, J8 Conn_01x09_Pin, J9 Conn_01x08_Pin

Commit message: Minor changes
Parts:
- removed J10, J12, J13, J15, J16, J5, J7, J9: Conn_01x08_Pin, Connector_PinHeader_2.54mm:PinHeader_1x08_P2.54mm_Vertical, symbol Connector:Conn_01x08_Pin
- removed J11, J14, J6, J8: Conn_01x09_Pin, Connector_PinHeader_2.54mm:PinHeader_1x09_P2.54mm_Vertical, symbol Connector:Conn_01x09_Pin
- added C106: .1u, Capacitor_SMD:C_0402_1005Metric, symbol Device:C_Small_US
- added J5, J6, J7, J8: Conn_01x25_Pin, Connector_PinHeader_2.54mm:PinHeader_1x25_P2.54mm_Vertical, symbol Connector:Conn_01x25_Pin
Connections:
- net 100_1: now also J5.1 (Pin_1)
- net 100_10: now also J6.5 (Pin_5)
- net 100_100: now also J8.25 (Pin_25)
- net 100_11: now also J5.6 (Pin_6)
- net 100_12: now also J6.6 (Pin_6)
- net 100_13: now also J5.7 (Pin_7)
- net 100_14: now also J6.7 (Pin_7)
- net 100_15: now also J5.8 (Pin_8)
- net 100_16: now also J6.8 (Pin_8)
- net 100_17: now also J5.9 (Pin_9)
- net 100_18: now also J6.9 (Pin_9)
- net 100_19: now also J5.10 (Pin_10)
- net 100_2: now also J6.1 (Pin_1)
- net 100_20: now also J6.10 (Pin_10)
- net 100_21: now also J5.11 (Pin_11)
- net 100_22: now also J6.11 (Pin_11)
- net 100_23: now also J5.12 (Pin_12)
- net 100_24: now also J6.12 (Pin_12)
- net 100_25: now also J5.13 (Pin_13)
- net 100_26: now also J6.13 (Pin_13)
- net 100_27: now also J5.14 (Pin_14)
- net 100_28: now also J6.14 (Pin_14)
- net 100_29: now also J5.15 (Pin_15)
- net 100_3: now also J5.2 (Pin_2)
- net 100_30: now also J6.15 (Pin_15)
- net 100_31: now also J5.16 (Pin_16)
- net 100_32: now also J6.16 (Pin_16)
- net 100_33: now also J5.17 (Pin_17)
- net 100_34: now also J6.17 (Pin_17)
- net 100_35: now also J5.18 (Pin_18)
- net 100_36: now also J6.18 (Pin_18)
- net 100_37: now also J5.19 (Pin_19)
- net 100_38: now also J6.19 (Pin_19)
- net 100_39: now also J5.20 (Pin_20)
- net 100_4: now also J6.2 (Pin_2)
- net 100_40: now also J6.20 (Pin_20)
- net 100_41: now also J5.21 (Pin_21)
- net 100_42: now also J6.21 (Pin_21)
- net 100_43: now also J5.22 (Pin_22)
- net 100_44: now also J6.22 (Pin_22)
- net 100_45: now also J5.23 (Pin_23)
- net 100_46: now also J6.23 (Pin_23)
- net 100_47: now also J5.24 (Pin_24)
- net 100_48: now also J6.24 (Pin_24)
- net 100_49: now also J5.25 (Pin_25)
- net 100_5: now also J5.3 (Pin_3)
- net 100_50: now also J6.25 (Pin_25)
- net 100_51: now also J7.1 (Pin_1)
- net 100_52: now also J8.1 (Pin_1)
- net 100_53: now also J7.2 (Pin_2)
- net 100_54: now also J8.2 (Pin_2)
- net 100_55: now also J7.3 (Pin_3)
- net 100_56: now also J8.3 (Pin_3)
- net 100_57: now also J7.4 (Pin_4)
- net 100_58: now also J8.4 (Pin_4)
- net 100_59: now also J7.5 (Pin_5)
- net 100_6: now also J6.3 (Pin_3)
- net 100_60: now also J8.5 (Pin_5)
- net 100_61: now also J7.6 (Pin_6)
- net 100_62: now also J8.6 (Pin_6)
- net 100_63: now also J7.7 (Pin_7)
- net 100_64: now also J8.7 (Pin_7)
- net 100_65: now also J7.8 (Pin_8)
- net 100_66: now also J8.8 (Pin_8)
- net 100_67: now also J7.9 (Pin_9)
- net 100_68: now also J8.9 (Pin_9)
- net 100_69: now also J7.10 (Pin_10)
- net 100_7: now also J5.4 (Pin_4)
- net 100_70: now also J8.10 (Pin_10)
- net 100_71: now also J7.11 (Pin_11)
- net 100_72: now also J4.7 (Pin_7), J_SOCKET_64_1.46, J8.11 (Pin_11)
- net 100_73: now also J7.12 (Pin_12)
- net 100_74: now also J8.12 (Pin_12)
- net 100_75: now also J7.13 (Pin_13)
- net 100_76: now also J3.9 (Pin_9), J_SOCKET_64_1.49, J8.13 (Pin_13)
- net 100_77: now also J7.14 (Pin_14)
- net 100_78: now also J8.14 (Pin_14)
- net 100_79: now also J7.15 (Pin_15)
- net 100_8: now also J6.4 (Pin_4)
- net 100_80: now also J8.15 (Pin_15)
- net 100_81: now also J7.16 (Pin_16)
- net 100_82: now also J8.16 (Pin_16)
- net 100_83: now also J7.17 (Pin_17)
- net 100_84: now also J8.17 (Pin_17)
- net 100_85: now also J7.18 (Pin_18)
- net 100_86: now also J8.18 (Pin_18)
- net 100_87: now also J7.19 (Pin_19)
- net 100_88: now also J8.19 (Pin_19)
- net 100_89: now also J7.20 (Pin_20)
- net 100_9: now also J5.5 (Pin_5)
- net 100_90: now also J8.20 (Pin_20)
- net 100_91: now also J7.21 (Pin_21)
- net 100_92: now also J8.21 (Pin_21)
- net 100_93: now also J7.22 (Pin_22)
- net 100_94: now also J8.22 (Pin_22)
- net 100_95: now also J7.23 (Pin_23)
- net 100_96: now also J8.23 (Pin_23)
- net 100_97: now also J7.24 (Pin_24)
- net 100_98: now also J8.24 (Pin_24)
- net 100_99: now also J7.25 (Pin_25)
- net 64_47: now also C106.1
- net GND: now also PARENT_DEAD1.G1 (GND1), PARENT_DEAD1.G2 (GND1__1), PARENT_DEAD1.G3 (GND1__2), PARENT_DEAD1.G4 (GND1__3), PARENT_DEAD1.G5 (GND2), PARENT_DEAD1.G6 (GND2__1), PARENT_DEAD1.G7 (GND2__2), PARENT_DEAD1.G8 (GND2__3), C106.2
- removed net 64_46: J4.7 (Pin_7), J_SOCKET_64_1.46, LQFP64_SWD1.1 (Pin_1)
- removed net 64_49: J3.9 (Pin_9), J_SOCKET_64_1.49, LQFP64_SWD1.2 (Pin_2)
- new net SWDCLK_64: LQFP64_SWD1.2 (Pin_2)
- new net SWDIO_64: LQFP64_SWD1.1 (Pin_1)
- no-connect marks 660 -> 652
Other:
- moved on the sheet: C100, C101, C102, C103, C104, C105, C96, C97, C98, C99, J1, J2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
